File: arisutea-pcb.kicad_pcb (KiCad board)
At the start: 2 copper layers, 339.1 x 121 mm, 182 parts, among them J12 VCC, J13 D+, J14 D-, J15 GND, J16 RGB, J17 RGB TO J18, J18 RGB FROM J17, J2 MISO, J3 +5V, J4 SCK, J5 MOSI, J6 ~RES~, J7 GND, SW1 SW_Push, SW10 SW_Push, SW11 SW_Push, SW12 SW_Push, SW13 SW_Push, SW14 SW_Push, SW15 SW_Push, SW16 SW_Push, SW17 SW_Push, SW18 SW_Push, SW19 SW_Push, SW2 SW_Push, SW20 SW_Push, SW21 SW_Push, SW22 SW_Push, SW23 SW_Push, SW24 SW_Push, SW25 SW_Push, SW26 SW_Push, SW27 SW_Push, SW28 SW_Push, SW29 SW_Push, SW3 SW_Push, SW30 SW_Push, SW31 SW_Push, SW32 SW_Push, SW33 SW_Push, SW34 SW_Push, SW35 SW_Push, SW36 SW_Push, SW37 SW_Push, SW38 SW_Push, SW39 SW_Push, SW4 SW_Push, SW40 SW_Push, SW41 SW_Push, SW42 SW_Push, SW43 SW_Push, SW44 SW_Push, SW45 SW_Push, SW46 SW_Push, SW47 SW_Push, SW48 SW_Push, SW49 SW_Push, SW5 SW_Push, SW50 SW_Push, SW51 SW_Push, SW52 SW_Push, SW53 SW_Push, SW54 SW_Push, SW55 SW_Push, SW56 SW_Push, SW57 SW_Push, SW58 SW_Push, SW59 SW_Push, SW6 SW_Push, SW60 SW_Push, SW61 SW_Push, SW62 SW_Push, SW63 SW_Push, SW64 SW_Push, SW65 SW_Push, SW66 SW_Push, SW7 SW_Push, SW8 SW_Push, SW9 SW_Push, U1 USBLC6-2SC6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

Commit message: housecleaning
Parts:
- added LOGO3: arisutea_logo, Symbol:OSHW-Logo_5.7x6mm_SilkScreen, F.Cu at (59.5, 111.3)
- added LOGO4: arisutea_logo, Symbol:OSHW-Logo_5.7x6mm_SilkScreen, B.Cu at (84.1, 111.2)
- added LOGO5: QMK_Logo_Light, 3x6_graphics:QMK_Logo_Light, F.Cu at (72.3, 119.1)
- added LOGO6: QMK_Logo_Light, 3x6_graphics:QMK_Logo_Light, B.Cu at (72.3, 119.1)
- J17: value RGB TO J18 -> RGB_IN
- J18: value RGB FROM J17 -> RGB_OUT
Connections:
- SW1 pad 1: Net-(D1-Pad2) -> /col0
- SW1 pad 2: /col0 -> Net-(D1-Pad2)
- SW10 pad 1: Net-(D10-Pad2) -> /col2
- SW10 pad 2: /col2 -> Net-(D10-Pad2)
- SW11 pad 1: Net-(D11-Pad2) -> /col2
- SW11 pad 2: /col2 -> Net-(D11-Pad2)
- SW12 pad 1: Net-(D12-Pad2) -> /col2
- SW12 pad 2: /col2 -> Net-(D12-Pad2)
- SW13 pad 1: Net-(D13-Pad2) -> /col2
- SW13 pad 2: /col2 -> Net-(D13-Pad2)
- SW14 pad 1: Net-(D14-Pad2) -> /col2
- SW14 pad 2: /col2 -> Net-(D14-Pad2)
- SW15 pad 1: Net-(D15-Pad2) -> /col3
- SW15 pad 2: /col3 -> Net-(D15-Pad2)
- SW16 pad 1: Net-(D16-Pad2) -> /col3
- SW16 pad 2: /col3 -> Net-(D16-Pad2)
- SW17 pad 1: Net-(D17-Pad2) -> /col3
- SW17 pad 2: /col3 -> Net-(D17-Pad2)
- SW18 pad 1: Net-(D18-Pad2) -> /col3
- SW18 pad 2: /col3 -> Net-(D18-Pad2)
- SW19 pad 1: Net-(D19-Pad2) -> /col4
- SW19 pad 2: /col4 -> Net-(D19-Pad2)
- SW2 pad 1: Net-(D2-Pad2) -> /col0
- SW2 pad 2: /col0 -> Net-(D2-Pad2)
- SW20 pad 1: Net-(D20-Pad2) -> /col4
- SW20 pad 2: /col4 -> Net-(D20-Pad2)
- SW21 pad 1: Net-(D21-Pad2) -> /col4
- SW21 pad 2: /col4 -> Net-(D21-Pad2)
- SW22 pad 1: Net-(D22-Pad2) -> /col4
- SW22 pad 2: /col4 -> Net-(D22-Pad2)
- SW23 pad 1: Net-(D23-Pad2) -> /col4
- SW23 pad 2: /col4 -> Net-(D23-Pad2)
- SW24 pad 1: Net-(D24-Pad2) -> /col5
- SW24 pad 2: /col5 -> Net-(D24-Pad2)
- SW25 pad 1: Net-(D25-Pad2) -> /col5
- SW25 pad 2: /col5 -> Net-(D25-Pad2)
- SW26 pad 1: Net-(D26-Pad2) -> /col5
- SW26 pad 2: /col5 -> Net-(D26-Pad2)
- SW27 pad 1: Net-(D27-Pad2) -> /col5
- SW27 pad 2: /col5 -> Net-(D27-Pad2)
- SW28 pad 1: Net-(D28-Pad2) -> /col5
- SW28 pad 2: /col5 -> Net-(D28-Pad2)
- SW29 pad 1: Net-(D29-Pad2) -> /col6
- SW29 pad 2: /col6 -> Net-(D29-Pad2)
- SW3 pad 1: Net-(D3-Pad2) -> /col0
- SW3 pad 2: /col0 -> Net-(D3-Pad2)
- SW30 pad 1: Net-(D30-Pad2) -> /col6
- SW30 pad 2: /col6 -> Net-(D30-Pad2)
- SW31 pad 1: Net-(D31-Pad2) -> /col6
- SW31 pad 2: /col6 -> Net-(D31-Pad2)
- SW32 pad 1: Net-(D32-Pad2) -> /col6
- SW32 pad 2: /col6 -> Net-(D32-Pad2)
- SW33 pad 1: Net-(D33-Pad2) -> /SCK
- SW33 pad 2: /SCK -> Net-(D33-Pad2)
- SW34 pad 1: Net-(D34-Pad2) -> /SCK
- SW34 pad 2: /SCK -> Net-(D34-Pad2)
- SW35 pad 1: Net-(D35-Pad2) -> /SCK
- SW35 pad 2: /SCK -> Net-(D35-Pad2)
- SW36 pad 1: Net-(D36-Pad2) -> /SCK
- SW36 pad 2: /SCK -> Net-(D36-Pad2)
- SW37 pad 1: Net-(D37-Pad2) -> /SCK
- SW37 pad 2: /SCK -> Net-(D37-Pad2)
- SW38 pad 1: Net-(D38-Pad2) -> /col8
- SW38 pad 2: /col8 -> Net-(D38-Pad2)
- SW39 pad 1: Net-(D39-Pad2) -> /col8
- SW39 pad 2: /col8 -> Net-(D39-Pad2)
- SW4 pad 1: Net-(D4-Pad2) -> /col0
- SW4 pad 2: /col0 -> Net-(D4-Pad2)
- SW40 pad 1: Net-(D40-Pad2) -> /col8
- SW40 pad 2: /col8 -> Net-(D40-Pad2)
- SW41 pad 1: Net-(D41-Pad2) -> /col8
- SW41 pad 2: /col8 -> Net-(D41-Pad2)
- SW42 pad 1: Net-(D42-Pad2) -> /col9
- SW42 pad 2: /col9 -> Net-(D42-Pad2)
- SW43 pad 1: Net-(D43-Pad2) -> /col9
- SW43 pad 2: /col9 -> Net-(D43-Pad2)
- SW44 pad 1: Net-(D44-Pad2) -> /col9
- SW44 pad 2: /col9 -> Net-(D44-Pad2)
- SW45 pad 1: Net-(D45-Pad2) -> /col9
- SW45 pad 2: /col9 -> Net-(D45-Pad2)
- SW46 pad 1: Net-(D46-Pad2) -> /col9
- SW46 pad 2: /col9 -> Net-(D46-Pad2)
- SW47 pad 1: Net-(D47-Pad2) -> /col10
- SW47 pad 2: /col10 -> Net-(D47-Pad2)
- SW48 pad 1: Net-(D48-Pad2) -> /col10
- SW48 pad 2: /col10 -> Net-(D48-Pad2)
- SW49 pad 1: Net-(D49-Pad2) -> /col10
- SW49 pad 2: /col10 -> Net-(D49-Pad2)
- SW5 pad 1: Net-(D5-Pad2) -> /col0
- SW5 pad 2: /col0 -> Net-(D5-Pad2)
- SW50 pad 1: Net-(D50-Pad2) -> /col10
- SW50 pad 2: /col10 -> Net-(D50-Pad2)
- SW51 pad 1: Net-(D51-Pad2) -> /col11
- SW51 pad 2: /col11 -> Net-(D51-Pad2)
- SW52 pad 1: Net-(D52-Pad2) -> /col11
- SW52 pad 2: /col11 -> Net-(D52-Pad2)
- SW53 pad 1: Net-(D53-Pad2) -> /col11
- SW53 pad 2: /col11 -> Net-(D53-Pad2)
- SW54 pad 1: Net-(D54-Pad2) -> /col11
- SW54 pad 2: /col11 -> Net-(D54-Pad2)
- SW55 pad 1: Net-(D55-Pad2) -> /col12
- SW55 pad 2: /col12 -> Net-(D55-Pad2)
- SW56 pad 1: Net-(D56-Pad2) -> /col12
- SW56 pad 2: /col12 -> Net-(D56-Pad2)
- SW57 pad 1: Net-(D57-Pad2) -> /col12
- SW57 pad 2: /col12 -> Net-(D57-Pad2)
- SW58 pad 1: Net-(D58-Pad2) -> /col12
- SW58 pad 2: /col12 -> Net-(D58-Pad2)
- SW59 pad 1: Net-(D59-Pad2) -> /col13
- SW59 pad 2: /col13 -> Net-(D59-Pad2)
- SW6 pad 1: Net-(D6-Pad2) -> /col1
- SW6 pad 2: /col1 -> Net-(D6-Pad2)
- SW60 pad 1: Net-(D60-Pad2) -> /col13
- SW60 pad 2: /col13 -> Net-(D60-Pad2)
- SW61 pad 1: Net-(D61-Pad2) -> /col13
- SW61 pad 2: /col13 -> Net-(D61-Pad2)
- SW62 pad 1: Net-(D62-Pad2) -> /col13
- SW62 pad 2: /col13 -> Net-(D62-Pad2)
- SW63 pad 1: Net-(D63-Pad2) -> /MISO
- SW63 pad 2: /MISO -> Net-(D63-Pad2)
- SW64 pad 1: Net-(D64-Pad2) -> /MISO
- SW64 pad 2: /MISO -> Net-(D64-Pad2)
- SW65 pad 1: Net-(D65-Pad2) -> /MISO
- SW65 pad 2: /MISO -> Net-(D65-Pad2)
- SW66 pad 1: Net-(D66-Pad2) -> /MISO
- SW66 pad 2: /MISO -> Net-(D66-Pad2)
- SW7 pad 1: Net-(D7-Pad2) -> /col1
- SW7 pad 2: /col1 -> Net-(D7-Pad2)
- SW8 pad 1: Net-(D8-Pad2) -> /col1
- SW8 pad 2: /col1 -> Net-(D8-Pad2)
- SW9 pad 1: Net-(D9-Pad2) -> /col1
- SW9 pad 2: /col1 -> Net-(D9-Pad2)

Commit message: underglow header placement moved a bit, add logos, move some components
Parts:
- LOGO3, LOGO4: footprint Symbol:OSHW-Logo_5.7x6mm_SilkScreen -> Symbol:OSHW-Logo_11.4x12mm_SilkScreen
- moved LOGO4 13.8 mm to (70.6, 114.2)
- moved LOGO3 11.5 mm to (70.6, 114.1)
- moved J16 11.2 mm to (31.6, 63.8)
- moved J18 10.5 mm to (354.9, 107.4), turned to 0 degrees
- moved J17 5.53 mm to (340.7, 57.9)
- moved LOGO5 4.55 mm to (70.4, 123.2)
- moved LOGO6 4.47 mm to (70.6, 123.2)
- moved C7 0.95 mm to (179.3, 53.8)
- moved R4 0.25 mm to (170.9, 52.1)
- renumbered LED2 to CAPS, LED1 to FN, LED3 to NUM
Routing:
- net RGB: track 170.4 -> 181.6 mm
- net +5V: track 312.4 -> 322.4 mm
- net GND: track 677.1 -> 670.4 mm
- net RGB_5V: track 50.8 -> 56.8 mm
- net /col8: track 108.1 -> 106.6 mm
- net /row2: track 406.1 -> 404.8 mm
- net /~RES~: track 40.7 -> 40.0 mm
- net /col13: track 297.6 -> 297.0 mm
- net /MOSI: track 40.0 -> 39.3 mm
- net RGB_A: track 50.8 -> 51.4 mm
- net /row1: track 388.9 -> 389.4 mm
- net /col12: vias 5 -> 4

Commit message: Initial upload of bluetooth version
Parts:
- removed C4: 1uF (±10%), arisutea:C_0805_2012Metric_Pad1.18x1.45mm_HandSolder
- removed C5: 1uF, arisutea:C_0805_2012Metric_Pad1.18x1.45mm_HandSolder
- removed C6, C7, C8, C9: 0.1uF, arisutea:C_0805_2012Metric_Pad1.18x1.45mm_HandSolder
- removed J12: VCC, arisutea:PinHeader_1x01_P2.54mm_Vertical
- removed J13: D+, arisutea:PinHeader_1x01_P2.54mm_Vertical
- removed J14: D-, arisutea:PinHeader_1x01_P2.54mm_Vertical
- removed J15, J7: GND, arisutea:PinHeader_1x01_P2.54mm_Vertical
- removed J16: RGB, arisutea:PinHeader_1x03_P2.54mm_Vertical
- removed J17: RGB_IN, arisutea:PinHeader_1x03_P2.54mm_Vertical
- removed J18: RGB_OUT, arisutea:PinHeader_1x03_P2.54mm_Vertical
- removed J2: MISO, arisutea:PinHeader_1x01_P2.54mm_Vertical
- removed J3: +5V, arisutea:PinHeader_1x01_P2.54mm_Vertical
- removed J4: SCK, arisutea:PinHeader_1x01_P2.54mm_Vertical
- removed J5: MOSI, arisutea:PinHeader_1x01_P2.54mm_Vertical
- removed J6: ~RES~, arisutea:PinHeader_1x01_P2.54mm_Vertical
- removed LOGO3, LOGO4: arisutea_logo, Symbol:OSHW-Logo_11.4x12mm_SilkScreen
- removed LOGO5, LOGO6: QMK_Logo_Light, 3x6_graphics:QMK_Logo_Light
- removed the R3 at (193.4, 28.8)
- removed the R4 at (170.9, 52.1)
- removed Y1: Crystal_GND24, arisutea:Crystal_SMD_TXC_7M-4Pin_3.2x2.5mm_HandSoldering
- added BT1: Battery_Cell, arisutea-bt-pcb:Battery_Connector, F.Cu at (156.0, 36.6)
- added BT2: Battery_Cell, arisutea-bt-pcb:JST_PH_S2B-PH-K_1x02_P2.00mm_Horizontal, B.Cu at (161.8, 37.2)
- added D1: 1N5819, arisutea-bt-pcb:D_SOD-123, B.Cu at (167.5, 70.0)
- added J1: Conn_01x04, arisutea-bt-pcb:PinHeader_1x04_P2.54mm_Vertical, F.Cu at (184.2, 106.2)
- added LED1: PWR_LED, arisutea-bt-pcb:LED_IN-S124ARUW, B.Cu at (193.0, 27.6)
- added LED5: BAT_LED, arisutea-bt-pcb:LED_IN-S124ARUW, B.Cu at (196.7, 27.6)
- added Q1: AO3401A, arisutea-bt-pcb:SOT-23, B.Cu at (164.6, 70.6)
- added R1: 5k1, arisutea-bt-pcb:R_0805_2012Metric_Pad1.20x1.40mm_HandSolder, B.Cu at (166.9, 26.3)
- added R10: 1K, arisutea-bt-pcb:R_0805_2012Metric_Pad1.20x1.40mm_HandSolder, B.Cu at (199.2, 27.6)
- added R2: 5k1, arisutea-bt-pcb:R_0805_2012Metric_Pad1.20x1.40mm_HandSolder, B.Cu at (184.3, 26.3)
- added R7: 10K, arisutea-bt-pcb:R_0805_2012Metric_Pad1.20x1.40mm_HandSolder, B.Cu at (171.8, 65.6)
- added R8: 1k, arisutea-bt-pcb:R_0805_2012Metric_Pad1.20x1.40mm_HandSolder, B.Cu at (190.4, 27.6)
- added R9: 10K, arisutea-bt-pcb:R_0805_2012Metric_Pad1.20x1.40mm_HandSolder, B.Cu at (184.2, 36.3)
- added SW67: Switch, arisutea-bt-pcb:OS102011MA1QN1, B.Cu at (157.0, 25.8)
- added U3: TP4504, arisutea-bt-pcb:SOT-23-5, B.Cu at (168.7, 65.7)
- added U4: AP2112K-3.3, arisutea-bt-pcb:SOT-23-5, B.Cu at (168.1, 74.5)
- C1: value 22pF -> 4.7uF; footprint arisutea:C_0805_2012Metric_Pad1.18x1.45mm_HandSolder -> arisutea-bt-pcb:C_0805_2012Metric_Pad1.18x1.45mm_HandSolder
- C2: value 22pF -> 1uF; footprint arisutea:C_0805_2012Metric_Pad1.18x1.45mm_HandSolder -> arisutea-bt-pcb:C_0805_2012Metric_Pad1.18x1.45mm_HandSolder
- C3: value 10uF -> 1uF; footprint arisutea:C_0805_2012Metric_Pad1.18x1.45mm_HandSolder -> arisutea-bt-pcb:C_0805_2012Metric_Pad1.18x1.45mm_HandSolder
- D10: renamed from D38; footprint arisutea:D_SOD-123 -> arisutea-bt-pcb:D_SOD-123
- D11: renamed from D42; footprint arisutea:D_SOD-123 -> arisutea-bt-pcb:D_SOD-123
- D12: renamed from D47; footprint arisutea:D_SOD-123 -> arisutea-bt-pcb:D_SOD-123
- D13: renamed from D51; footprint arisutea:D_SOD-123 -> arisutea-bt-pcb:D_SOD-123
- D14: renamed from D55; footprint arisutea:D_SOD-123 -> arisutea-bt-pcb:D_SOD-123
- D15: renamed from D59; footprint arisutea:D_SOD-123 -> arisutea-bt-pcb:D_SOD-123
- D16: renamed from D2; footprint arisutea:D_SOD-123 -> arisutea-bt-pcb:D_SOD-123
- D17: renamed from D7; footprint arisutea:D_SOD-123 -> arisutea-bt-pcb:D_SOD-123
- D18: renamed from D11; footprint arisutea:D_SOD-123 -> arisutea-bt-pcb:D_SOD-123
- D19: renamed from D16; footprint arisutea:D_SOD-123 -> arisutea-bt-pcb:D_SOD-123
- D2: renamed from D1; footprint arisutea:D_SOD-123 -> arisutea-bt-pcb:D_SOD-123
- D20: footprint arisutea:D_SOD-123 -> arisutea-bt-pcb:D_SOD-123
- D21: renamed from D25; footprint arisutea:D_SOD-123 -> arisutea-bt-pcb:D_SOD-123
- D22: renamed from D30; footprint arisutea:D_SOD-123 -> arisutea-bt-pcb:D_SOD-123
- D23: renamed from D34; footprint arisutea:D_SOD-123 -> arisutea-bt-pcb:D_SOD-123
- D24: renamed from D39; footprint arisutea:D_SOD-123 -> arisutea-bt-pcb:D_SOD-123
- D25: renamed from D43; footprint arisutea:D_SOD-123 -> arisutea-bt-pcb:D_SOD-123
- D26: renamed from D48; footprint arisutea:D_SOD-123 -> arisutea-bt-pcb:D_SOD-123
- D27: renamed from D52; footprint arisutea:D_SOD-123 -> arisutea-bt-pcb:D_SOD-123
- D28: renamed from D56; footprint arisutea:D_SOD-123 -> arisutea-bt-pcb:D_SOD-123
- D29: renamed from D60; footprint arisutea:D_SOD-123 -> arisutea-bt-pcb:D_SOD-123
- D3: renamed from D6; footprint arisutea:D_SOD-123 -> arisutea-bt-pcb:D_SOD-123
- D30: renamed from D63; footprint arisutea:D_SOD-123 -> arisutea-bt-pcb:D_SOD-123
- D31: renamed from D3; footprint arisutea:D_SOD-123 -> arisutea-bt-pcb:D_SOD-123
- D32: renamed from D8; footprint arisutea:D_SOD-123 -> arisutea-bt-pcb:D_SOD-123
- D33: renamed from D12; footprint arisutea:D_SOD-123 -> arisutea-bt-pcb:D_SOD-123
- D34: renamed from D17; footprint arisutea:D_SOD-123 -> arisutea-bt-pcb:D_SOD-123
- D35: renamed from D21; footprint arisutea:D_SOD-123 -> arisutea-bt-pcb:D_SOD-123
- D36: renamed from D26; footprint arisutea:D_SOD-123 -> arisutea-bt-pcb:D_SOD-123
- D37: renamed from D31; footprint arisutea:D_SOD-123 -> arisutea-bt-pcb:D_SOD-123
- D38: renamed from D35; footprint arisutea:D_SOD-123 -> arisutea-bt-pcb:D_SOD-123
- D39: renamed from D40; footprint arisutea:D_SOD-123 -> arisutea-bt-pcb:D_SOD-123
- D4: renamed from D10; footprint arisutea:D_SOD-123 -> arisutea-bt-pcb:D_SOD-123
- D40: renamed from D44; footprint arisutea:D_SOD-123 -> arisutea-bt-pcb:D_SOD-123
- D41: renamed from D49; footprint arisutea:D_SOD-123 -> arisutea-bt-pcb:D_SOD-123
- D42: renamed from D53; footprint arisutea:D_SOD-123 -> arisutea-bt-pcb:D_SOD-123
- D43: renamed from D57; footprint arisutea:D_SOD-123 -> arisutea-bt-pcb:D_SOD-123
- D44: renamed from D64; footprint arisutea:D_SOD-123 -> arisutea-bt-pcb:D_SOD-123
- D45: renamed from D4; footprint arisutea:D_SOD-123 -> arisutea-bt-pcb:D_SOD-123
- D46: renamed from D9; footprint arisutea:D_SOD-123 -> arisutea-bt-pcb:D_SOD-123
- D47: renamed from D13; footprint arisutea:D_SOD-123 -> arisutea-bt-pcb:D_SOD-123
- D48: renamed from D18; footprint arisutea:D_SOD-123 -> arisutea-bt-pcb:D_SOD-123
- D49: renamed from D22; footprint arisutea:D_SOD-123 -> arisutea-bt-pcb:D_SOD-123
- D5: renamed from D15; footprint arisutea:D_SOD-123 -> arisutea-bt-pcb:D_SOD-123
- D50: renamed from D27; footprint arisutea:D_SOD-123 -> arisutea-bt-pcb:D_SOD-123
- D51: renamed from D32; footprint arisutea:D_SOD-123 -> arisutea-bt-pcb:D_SOD-123
- D52: renamed from D36; footprint arisutea:D_SOD-123 -> arisutea-bt-pcb:D_SOD-123
- D53: renamed from D41; footprint arisutea:D_SOD-123 -> arisutea-bt-pcb:D_SOD-123
- D54: renamed from D45; footprint arisutea:D_SOD-123 -> arisutea-bt-pcb:D_SOD-123
- D55: renamed from D50; footprint arisutea:D_SOD-123 -> arisutea-bt-pcb:D_SOD-123
- D56: renamed from D54; footprint arisutea:D_SOD-123 -> arisutea-bt-pcb:D_SOD-123
- D57: renamed from D61; footprint arisutea:D_SOD-123 -> arisutea-bt-pcb:D_SOD-123
- D58: renamed from D65; footprint arisutea:D_SOD-123 -> arisutea-bt-pcb:D_SOD-123
- D59: renamed from D5; footprint arisutea:D_SOD-123 -> arisutea-bt-pcb:D_SOD-123
- D6: renamed from D19; footprint arisutea:D_SOD-123 -> arisutea-bt-pcb:D_SOD-123
- D60: renamed from D14; footprint arisutea:D_SOD-123 -> arisutea-bt-pcb:D_SOD-123
- D61: renamed from D23; footprint arisutea:D_SOD-123 -> arisutea-bt-pcb:D_SOD-123
- D62: renamed from D28; footprint arisutea:D_SOD-123 -> arisutea-bt-pcb:D_SOD-123
- D63: renamed from D37; footprint arisutea:D_SOD-123 -> arisutea-bt-pcb:D_SOD-123
- D64: renamed from D46; footprint arisutea:D_SOD-123 -> arisutea-bt-pcb:D_SOD-123
- D65: renamed from D58; footprint arisutea:D_SOD-123 -> arisutea-bt-pcb:D_SOD-123
- D66: renamed from D62; footprint arisutea:D_SOD-123 -> arisutea-bt-pcb:D_SOD-123
- D67: renamed from D66; footprint arisutea:D_SOD-123 -> arisutea-bt-pcb:D_SOD-123
- D7: renamed from D24; footprint arisutea:D_SOD-123 -> arisutea-bt-pcb:D_SOD-123
- D8: renamed from D29; footprint arisutea:D_SOD-123 -> arisutea-bt-pcb:D_SOD-123
- D9: renamed from D33; footprint arisutea:D_SOD-123 -> arisutea-bt-pcb:D_SOD-123
- F1: footprint arisutea:Fuse_1206_3216Metric_Pad1.42x1.75mm_HandSolder -> arisutea-bt-pcb:Fuse_1206_3216Metric_Pad1.42x1.75mm_HandSolder
- H1, H2, H3, H4, H5, H6, H7, H8: footprint arisutea:Plated_Through_Hole_M2 -> arisutea-bt-pcb:Generic-Mounthole
- LED2: renamed from FN; footprint arisutea:LED_IN-S124ARUW -> arisutea-bt-pcb:LED_IN-S124ARUW
- LED3: renamed from CAPS; footprint arisutea:LED_IN-S124ARUW -> arisutea-bt-pcb:LED_IN-S124ARUW
- LED4: renamed from NUM; footprint arisutea:LED_IN-S124ARUW -> arisutea-bt-pcb:LED_IN-S124ARUW
- LOGO1, LOGO2: value arisutea_logo -> LOGO; footprint arisutea:arisutea_logo -> arisutea-bt-pcb:arisutea_logo
- R11: renamed from R7; footprint arisutea:R_0805_2012Metric_Pad1.20x1.40mm_HandSolder -> arisutea-bt-pcb:R_0805_2012Metric_Pad1.20x1.40mm_HandSolder
- R12: renamed from R8; footprint arisutea:R_0805_2012Metric_Pad1.20x1.40mm_HandSolder -> arisutea-bt-pcb:R_0805_2012Metric_Pad1.20x1.40mm_HandSolder
- R13: renamed from R9; footprint arisutea:R_0805_2012Metric_Pad1.20x1.40mm_HandSolder -> arisutea-bt-pcb:R_0805_2012Metric_Pad1.20x1.40mm_HandSolder
- R3: renamed from R2; footprint arisutea:R_0805_2012Metric_Pad1.20x1.40mm_HandSolder -> arisutea-bt-pcb:R_0805_2012Metric_Pad1.20x1.40mm_HandSolder
- R4: renamed from R1; footprint arisutea:R_0805_2012Metric_Pad1.20x1.40mm_HandSolder -> arisutea-bt-pcb:R_0805_2012Metric_Pad1.20x1.40mm_HandSolder
- R5: value 5k1 -> 806K; footprint arisutea:R_0805_2012Metric_Pad1.20x1.40mm_HandSolder -> arisutea-bt-pcb:R_0805_2012Metric_Pad1.20x1.40mm_HandSolder
- R6: value 5k1 -> 2M; footprint arisutea:R_0805_2012Metric_Pad1.20x1.40mm_HandSolder -> arisutea-bt-pcb:R_0805_2012Metric_Pad1.20x1.40mm_HandSolder
- SW1, SW66: footprint arisutea:SW_Hotswap_Kailh_1.00u -> arisutea-bt-pcb:SW_Hotswap_Kailh_1.00u
- SW10: renamed from SW42; footprint arisutea:SW_Hotswap_Kailh_1.00u -> arisutea-bt-pcb:SW_Hotswap_Kailh_1.00u
- SW11: renamed from SW47; footprint arisutea:SW_Hotswap_Kailh_1.00u -> arisutea-bt-pcb:SW_Hotswap_Kailh_1.00u
- SW12: renamed from SW51; footprint arisutea:SW_Hotswap_Kailh_1.00u -> arisutea-bt-pcb:SW_Hotswap_Kailh_1.00u
- SW13: renamed from SW55; footprint arisutea:SW_Hotswap_Kailh_1.00u -> arisutea-bt-pcb:SW_Hotswap_Kailh_1.00u
- SW14: renamed from SW59; footprint arisutea:SW_Hotswap_Kailh_2.00u -> arisutea-bt-pcb:SW_Hotswap_Kailh_2.00u
- SW15: renamed from SW2; footprint arisutea:SW_Hotswap_Kailh_1.50u -> arisutea-bt-pcb:SW_Hotswap_Kailh_1.50u
- SW16: renamed from SW7; footprint arisutea:SW_Hotswap_Kailh_1.00u -> arisutea-bt-pcb:SW_Hotswap_Kailh_1.00u
- SW17: renamed from SW11; footprint arisutea:SW_Hotswap_Kailh_1.00u -> arisutea-bt-pcb:SW_Hotswap_Kailh_1.00u
- SW18: renamed from SW16; footprint arisutea:SW_Hotswap_Kailh_1.00u -> arisutea-bt-pcb:SW_Hotswap_Kailh_1.00u
- SW19: renamed from SW20; footprint arisutea:SW_Hotswap_Kailh_1.00u -> arisutea-bt-pcb:SW_Hotswap_Kailh_1.00u
- SW2: renamed from SW6; footprint arisutea:SW_Hotswap_Kailh_1.00u -> arisutea-bt-pcb:SW_Hotswap_Kailh_1.00u
- SW20: renamed from SW25; footprint arisutea:SW_Hotswap_Kailh_1.00u -> arisutea-bt-pcb:SW_Hotswap_Kailh_1.00u
- SW21: renamed from SW30; footprint arisutea:SW_Hotswap_Kailh_1.00u -> arisutea-bt-pcb:SW_Hotswap_Kailh_1.00u
- SW22: renamed from SW34; footprint arisutea:SW_Hotswap_Kailh_1.00u -> arisutea-bt-pcb:SW_Hotswap_Kailh_1.00u
- SW23: renamed from SW39; footprint arisutea:SW_Hotswap_Kailh_1.00u -> arisutea-bt-pcb:SW_Hotswap_Kailh_1.00u
- SW24: renamed from SW43; footprint arisutea:SW_Hotswap_Kailh_1.00u -> arisutea-bt-pcb:SW_Hotswap_Kailh_1.00u
- SW25: renamed from SW48; footprint arisutea:SW_Hotswap_Kailh_1.00u -> arisutea-bt-pcb:SW_Hotswap_Kailh_1.00u
- SW26: renamed from SW52; footprint arisutea:SW_Hotswap_Kailh_1.00u -> arisutea-bt-pcb:SW_Hotswap_Kailh_1.00u
- SW27: renamed from SW56; footprint arisutea:SW_Hotswap_Kailh_1.00u -> arisutea-bt-pcb:SW_Hotswap_Kailh_1.00u
- SW28: renamed from SW60; footprint arisutea:SW_Hotswap_Kailh_1.50u -> arisutea-bt-pcb:SW_Hotswap_Kailh_1.50u
- SW29: renamed from SW63; footprint arisutea:SW_Hotswap_Kailh_1.00u -> arisutea-bt-pcb:SW_Hotswap_Kailh_1.00u
- SW3: renamed from SW10; footprint arisutea:SW_Hotswap_Kailh_1.00u -> arisutea-bt-pcb:SW_Hotswap_Kailh_1.00u
- SW30: renamed from SW3; footprint arisutea:SW_Hotswap_Kailh_1.75u -> arisutea-bt-pcb:SW_Hotswap_Kailh_1.75u
- SW31: renamed from SW8; footprint arisutea:SW_Hotswap_Kailh_1.00u -> arisutea-bt-pcb:SW_Hotswap_Kailh_1.00u
- SW32: renamed from SW12; footprint arisutea:SW_Hotswap_Kailh_1.00u -> arisutea-bt-pcb:SW_Hotswap_Kailh_1.00u
- SW33: renamed from SW17; footprint arisutea:SW_Hotswap_Kailh_1.00u -> arisutea-bt-pcb:SW_Hotswap_Kailh_1.00u
- SW34: renamed from SW21; footprint arisutea:SW_Hotswap_Kailh_1.00u -> arisutea-bt-pcb:SW_Hotswap_Kailh_1.00u
- SW35: renamed from SW26; footprint arisutea:SW_Hotswap_Kailh_1.00u -> arisutea-bt-pcb:SW_Hotswap_Kailh_1.00u
- SW36: renamed from SW31; footprint arisutea:SW_Hotswap_Kailh_1.00u -> arisutea-bt-pcb:SW_Hotswap_Kailh_1.00u
- SW37: renamed from SW35; footprint arisutea:SW_Hotswap_Kailh_1.00u -> arisutea-bt-pcb:SW_Hotswap_Kailh_1.00u
- SW38: renamed from SW40; footprint arisutea:SW_Hotswap_Kailh_1.00u -> arisutea-bt-pcb:SW_Hotswap_Kailh_1.00u
- SW39: renamed from SW44; footprint arisutea:SW_Hotswap_Kailh_1.00u -> arisutea-bt-pcb:SW_Hotswap_Kailh_1.00u
- SW4: renamed from SW15; footprint arisutea:SW_Hotswap_Kailh_1.00u -> arisutea-bt-pcb:SW_Hotswap_Kailh_1.00u
- SW40: renamed from SW49; footprint arisutea:SW_Hotswap_Kailh_1.00u -> arisutea-bt-pcb:SW_Hotswap_Kailh_1.00u
- SW41: renamed from SW53; footprint arisutea:SW_Hotswap_Kailh_1.00u -> arisutea-bt-pcb:SW_Hotswap_Kailh_1.00u
- SW42: renamed from SW57; footprint arisutea:SW_Hotswap_Kailh_2.25u_RevStab -> arisutea-bt-pcb:SW_Hotswap_Kailh_2.25u_RevStab
- SW43: renamed from SW64; footprint arisutea:SW_Hotswap_Kailh_1.00u -> arisutea-bt-pcb:SW_Hotswap_Kailh_1.00u
- SW44: renamed from SW4; footprint arisutea:SW_Hotswap_Kailh_2.25u -> arisutea-bt-pcb:SW_Hotswap_Kailh_2.25u
- SW45: renamed from SW9; footprint arisutea:SW_Hotswap_Kailh_1.00u -> arisutea-bt-pcb:SW_Hotswap_Kailh_1.00u
- SW46: renamed from SW13; footprint arisutea:SW_Hotswap_Kailh_1.00u -> arisutea-bt-pcb:SW_Hotswap_Kailh_1.00u
- SW47: renamed from SW18; footprint arisutea:SW_Hotswap_Kailh_1.00u -> arisutea-bt-pcb:SW_Hotswap_Kailh_1.00u
- SW48: renamed from SW22; footprint arisutea:SW_Hotswap_Kailh_1.00u -> arisutea-bt-pcb:SW_Hotswap_Kailh_1.00u
- SW49: renamed from SW27; footprint arisutea:SW_Hotswap_Kailh_1.00u -> arisutea-bt-pcb:SW_Hotswap_Kailh_1.00u
- SW5: renamed from SW19; footprint arisutea:SW_Hotswap_Kailh_1.00u -> arisutea-bt-pcb:SW_Hotswap_Kailh_1.00u
- SW50: renamed from SW32; footprint arisutea:SW_Hotswap_Kailh_1.00u -> arisutea-bt-pcb:SW_Hotswap_Kailh_1.00u
- SW51: renamed from SW36; footprint arisutea:SW_Hotswap_Kailh_1.00u -> arisutea-bt-pcb:SW_Hotswap_Kailh_1.00u
- SW52: renamed from SW41; footprint arisutea:SW_Hotswap_Kailh_1.00u -> arisutea-bt-pcb:SW_Hotswap_Kailh_1.00u
- SW53: renamed from SW45; footprint arisutea:SW_Hotswap_Kailh_1.00u -> arisutea-bt-pcb:SW_Hotswap_Kailh_1.00u
- SW54: renamed from SW50; footprint arisutea:SW_Hotswap_Kailh_1.00u -> arisutea-bt-pcb:SW_Hotswap_Kailh_1.00u
- SW55: renamed from SW54; footprint arisutea:SW_Hotswap_Kailh_1.75u -> arisutea-bt-pcb:SW_Hotswap_Kailh_1.75u
- SW56: renamed from SW61; footprint arisutea:SW_Hotswap_Kailh_1.00u -> arisutea-bt-pcb:SW_Hotswap_Kailh_1.00u
- SW57: renamed from SW65; footprint arisutea:SW_Hotswap_Kailh_1.00u -> arisutea-bt-pcb:SW_Hotswap_Kailh_1.00u
- SW58: renamed from SW5; footprint arisutea:SW_Hotswap_Kailh_1.50u -> arisutea-bt-pcb:SW_Hotswap_Kailh_1.50u
- SW59: renamed from SW14; footprint arisutea:SW_Hotswap_Kailh_1.00u -> arisutea-bt-pcb:SW_Hotswap_Kailh_1.00u
- SW6: renamed from SW24; footprint arisutea:SW_Hotswap_Kailh_1.00u -> arisutea-bt-pcb:SW_Hotswap_Kailh_1.00u
- SW60: renamed from SW23; footprint arisutea:SW_Hotswap_Kailh_2.00u_RevStab -> arisutea-bt-pcb:SW_Hotswap_Kailh_2.00u_RevStab
- SW61: renamed from SW28; footprint arisutea:SW_Hotswap_Kailh_1.00u -> arisutea-bt-pcb:SW_Hotswap_Kailh_1.00u
- SW62: renamed from SW37; footprint arisutea:SW_Hotswap_Kailh_2.75u_RevStab -> arisutea-bt-pcb:SW_Hotswap_Kailh_2.75u_RevStab
- SW63: renamed from SW46; footprint arisutea:SW_Hotswap_Kailh_1.00u -> arisutea-bt-pcb:SW_Hotswap_Kailh_1.00u
- SW64: renamed from SW58; footprint arisutea:SW_Hotswap_Kailh_1.00u -> arisutea-bt-pcb:SW_Hotswap_Kailh_1.00u
- SW65: renamed from SW62; footprint arisutea:SW_Hotswap_Kailh_1.00u -> arisutea-bt-pcb:SW_Hotswap_Kailh_1.00u
- SW7: renamed from SW29; footprint arisutea:SW_Hotswap_Kailh_1.00u -> arisutea-bt-pcb:SW_Hotswap_Kailh_1.00u
- SW8: renamed from SW33; footprint arisutea:SW_Hotswap_Kailh_1.00u -> arisutea-bt-pcb:SW_Hotswap_Kailh_1.00u
- SW9: renamed from SW38; footprint arisutea:SW_Hotswap_Kailh_1.00u -> arisutea-bt-pcb:SW_Hotswap_Kailh_1.00u
- SWR1: footprint arisutea:SW_SPST_TL3342 -> arisutea-bt-pcb:SW_SPST_TL3342
- U1: value USBLC6-2SC6 -> nRF52840_holyiot_18010; footprint arisutea:SOT-23-6_Handsoldering -> arisutea-bt-pcb:nRF52840_holyiot_18010_HS_simple
- U2: value ATmega32U4-AU -> USBLC6-2SC6; footprint arisutea:TQFP-44_10x10mm_P0.8mm -> arisutea-bt-pcb:SOT-23-6_Handsoldering
- USB1: value USB_C_HRO_TYPE-C-31-M-12-USB_Type-C -> HRO-TYPE-C-31-M-12-Type-C; footprint arisutea:USB_C_Receptacle_HRO_TYPE-C-31-M-12-HandSoldering -> arisutea-bt-pcb:USB_C_Receptacle_HRO_TYPE-C-31-M-12-HandSoldering
- moved U1 58.4 mm to (167.9, 89.3), turned to 0 degrees
- moved SWR1 53.2 mm to (147.1, 28.0)
- moved C2 47.1 mm to (161.3, 78.4), turned to 180 degrees
- moved C3 43.6 mm to (169.8, 70.4)
- moved R5 43.6 mm to (163.4, 74.3)
- moved R6 38.5 mm to (165.3, 74.3), turned to 270 degrees
- moved C1 31.4 mm to (164.7, 64.9), turned to 180 degrees
- moved F1 23.3 mm to (183.7, 32.6)
- moved R4 19.0 mm to (176.5, 41.2), turned to 90 degrees
- moved R3 18.6 mm to (174.5, 41.2), turned to 90 degrees
- moved U2 7.05 mm to (175.5, 35.1)
- moved USB1 3.77 mm to (175.5, 24.5)
- moved H5 0.31 mm to (229.2, 28.2)
- moved H1 0.06 mm to (56.8, 48.3)
- turned LED2 to 90 degrees
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Connections:
- C1 pad 2: XTAL1 -> vbat
- C2 pad 1: XTAL2 -> VDD_nRF
- C3 pad 1: +5V -> Net-(C3-Pad1)
- D10 pad 1: /row0 -> row0
- D11 pad 1: /row0 -> row0
- D12 pad 1: /row0 -> row0
- D13 pad 1: /row0 -> row0
- D14 pad 1: /row0 -> row0
- D15 pad 1: /row0 -> row0
- D16 pad 1: /row1 -> row1
- D17 pad 1: /row1 -> row1
- D18 pad 1: /row1 -> row1
- D19 pad 1: /row1 -> row1
- D2 pad 1: /row0 -> row0
- D20 pad 1: /row1 -> row1
- D21 pad 1: /row1 -> row1
- D22 pad 1: /row1 -> row1
- D23 pad 1: /row1 -> row1
- D24 pad 1: /row1 -> row1
- D25 pad 1: /row1 -> row1
- D26 pad 1: /row1 -> row1
- D27 pad 1: /row1 -> row1
- D28 pad 1: /row1 -> row1
- D29 pad 1: /row1 -> row1
- D3 pad 1: /row0 -> row0
- D30 pad 1: /row1 -> row1
- D31 pad 1: /row2 -> row2
- D32 pad 1: /row2 -> row2
- D33 pad 1: /row2 -> row2
- D34 pad 1: /row2 -> row2
- D35 pad 1: /row2 -> row2
- D36 pad 1: /row2 -> row2
- D37 pad 1: /row2 -> row2
- D38 pad 1: /row2 -> row2
- D39 pad 1: /row2 -> row2
- D4 pad 1: /row0 -> row0
- D40 pad 1: /row2 -> row2
- D41 pad 1: /row2 -> row2
- D42 pad 1: /row2 -> row2
- D43 pad 1: /row2 -> row2
- D44 pad 1: /row2 -> row2
- D45 pad 1: /row3 -> row3
- D46 pad 1: /row3 -> row3
- D47 pad 1: /row3 -> row3
- D48 pad 1: /row3 -> row3
- D49 pad 1: /row3 -> row3
- D5 pad 1: /row0 -> row0
- D50 pad 1: /row3 -> row3
- D51 pad 1: /row3 -> row3
- D52 pad 1: /row3 -> row3
- D53 pad 1: /row3 -> row3
- D54 pad 1: /row3 -> row3
- D55 pad 1: /row3 -> row3
- D56 pad 1: /row3 -> row3
- D57 pad 1: /row3 -> row3
- D58 pad 1: /row3 -> row3
- D59 pad 1: /row4 -> row4
- D6 pad 1: /row0 -> row0
- D60 pad 1: /row4 -> row4
- D61 pad 1: /row4 -> row4
- D62 pad 1: /row4 -> row4
- D63 pad 1: /row4 -> row4
- D64 pad 1: /row4 -> row4
- D65 pad 1: /row4 -> row4
- D66 pad 1: /row4 -> row4
- D67 pad 1: /row4 -> row4
- D7 pad 1: /row0 -> row0
- D8 pad 1: /row0 -> row0
- D9 pad 1: /row0 -> row0
- F1 pad 1: +5V -> vbus_usb
- F1 pad 2: VCC -> VBUS
- R3 pad 2: Net-(J14-Pad1) -> Net-(R3-Pad2)
- R4 pad 2: Net-(J13-Pad1) -> Net-(R4-Pad2)
- R5 pad 1: Net-(R5-Pad1) -> bat_volt
- R5 pad 2: GND -> vbat
- R6 pad 1: Net-(R6-Pad1) -> GND
- R6 pad 2: GND -> bat_volt
- SW1 pad 1: /col0 -> col0
- SW10 pad 1: /col9 -> col9
- SW11 pad 1: /col10 -> col10
- SW12 pad 1: /col11 -> col11
- SW13 pad 1: /col12 -> col12
- SW14 pad 1: /col13 -> col13
- SW15 pad 1: /col0 -> col0
- SW16 pad 1: /col1 -> col1
- SW17 pad 1: /col2 -> col2
- SW18 pad 1: /col3 -> col3
- SW19 pad 1: /col4 -> col4
- SW2 pad 1: /col1 -> col1
- SW20 pad 1: /col5 -> col5
- SW21 pad 1: /col6 -> col6
- SW22 pad 1: /SCK -> col7
- SW23 pad 1: /col8 -> col8
- SW24 pad 1: /col9 -> col9
- SW25 pad 1: /col10 -> col10
- SW26 pad 1: /col11 -> col11
- SW27 pad 1: /col12 -> col12
- SW28 pad 1: /col13 -> col13
- SW29 pad 1: /MISO -> col14
- SW3 pad 1: /col2 -> col2
- SW30 pad 1: /col0 -> col0
- SW31 pad 1: /col1 -> col1
- SW32 pad 1: /col2 -> col2
- SW33 pad 1: /col3 -> col3
- SW34 pad 1: /col4 -> col4
- SW35 pad 1: /col5 -> col5
- SW36 pad 1: /col6 -> col6
- SW37 pad 1: /SCK -> col7
- SW38 pad 1: /col8 -> col8
- SW39 pad 1: /col9 -> col9
- SW4 pad 1: /col3 -> col3
- SW40 pad 1: /col10 -> col10
- SW41 pad 1: /col11 -> col11
- SW42 pad 1: /col12 -> col12
- SW43 pad 1: /MISO -> col14
- SW44 pad 1: /col0 -> col0
- SW45 pad 1: /col1 -> col1
- SW46 pad 1: /col2 -> col2
- SW47 pad 1: /col3 -> col3
- SW48 pad 1: /col4 -> col4
- SW49 pad 1: /col5 -> col5
- SW5 pad 1: /col4 -> col4
- SW50 pad 1: /col6 -> col6
- SW51 pad 1: /SCK -> col7
- SW52 pad 1: /col8 -> col8
- SW53 pad 1: /col9 -> col9
- SW54 pad 1: /col10 -> col10
- SW55 pad 1: /col11 -> col11
- SW56 pad 1: /col13 -> col13
- SW57 pad 1: /MISO -> col14
- SW58 pad 1: /col0 -> col0
- SW59 pad 1: /col2 -> col2
- SW6 pad 1: /col5 -> col5
- SW60 pad 1: /col4 -> col4
- SW61 pad 1: /col5 -> col5
- SW62 pad 1: /SCK -> col7
- SW63 pad 1: /col9 -> col9
- SW64 pad 1: /col12 -> col12
- SW65 pad 1: /col13 -> col13
- SW66 pad 1: /MISO -> col14
- SW7 pad 1: /col6 -> col6
- SW8 pad 1: /SCK -> col7
- SW9 pad 1: /col8 -> col8
- SWR1 pad 2: /~RES~ -> reset
- U1 pad 1: Net-(U1-Pad1) -> GND
- U1 pad 2: GND -> Net-(U1-Pad2)
- U1 pad 3: Net-(U1-Pad3) -> row3
- U1 pad 4: Net-(J13-Pad1) -> row4
- U1 pad 5: VCC -> row2
- U1 pad 6: Net-(J14-Pad1) -> Net-(U1-Pad6)
- U2 pad 1: /col2 -> Net-(U2-Pad1)
- U2 pad 2: +5V -> GND
- U2 pad 3: D- -> Net-(U2-Pad3)
- U2 pad 4: D+ -> Net-(R4-Pad2)
- U2 pad 5: GND -> vbus_usb
- U2 pad 6: Net-(C4-Pad1) -> Net-(R3-Pad2)
Routing:
- net GND: track 670.4 -> 103.8 mm
- net /row3: track 442.5 -> 0.00 mm, vias 2 -> 0
- net /row4: track 434.3 -> 0.00 mm, vias 2 -> 0
- net /row2: track 404.8 -> 0.00 mm, vias 2 -> 0
- net /row1: track 389.4 -> 0.00 mm, vias 4 -> 0
- net row3: track 0.00 -> 376.2 mm, vias 0 -> 2
- net row4: track 0.00 -> 376.1 mm, vias 0 -> 2
- net row1: track 0.00 -> 338.5 mm, vias 0 -> 2
- net row2: track 0.00 -> 335.6 mm, vias 0 -> 2
- net /row0: track 324.2 -> 0.00 mm, vias 4 -> 0
- net +5V: track 322.4 -> 0.00 mm, vias 7 -> 0
- net row0: track 0.00 -> 310.2 mm, vias 0 -> 2
- net /col12: track 298.9 -> 0.00 mm, vias 4 -> 0
- net /col13: track 297.0 -> 0.00 mm, vias 5 -> 0
- net col14: track 0.00 -> 286.3 mm, vias 0 -> 5
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Other:
- outline, holes or cut-outs redrawn
- net class Comms added: clearance 0.127, trace_width 0.25, via_dia 0.6, via_drill 0.3
- net class Default: trace_width 0.254 -> 0.25; via_dia 0.8 -> 0.6; via_drill 0.4 -> 0.3
- net class Power removed
- net class Power 1.5A added: clearance 0.127, trace_width 0.4, via_dia 0.6, via_drill 0.4
- net class Power 3A added: clearance 0.127, trace_width 0.55, via_dia 0.9, via_drill 0.6
- net class Power Input added: clearance 0.127, trace_width 0.45, via_dia 0.6, via_drill 0.3
- net class Tight added: clearance 0.127, trace_width 0.127, via_dia 0.6, via_drill 0.3
- board text added: "Arisutea-BT Rev 0.1 3x6 Design mattyams"
- board text removed: "+5V"
- board text removed: "Arisutea Rev 0.6 3x6 Design mattyams"
- board text removed: "DATA"
- board text removed: "GND"
