File: arisutea-pcb.sch (KiCad schematic (older format))
At the start: 54 parts, among them J12 VCC, J13 D+, J14 D-, J15 GND, J16 RGB, J17 RGB_IN, J18 RGB_OUT, J2 MISO, J3 +5V, J4 SCK, J5 MOSI, J6 ~RES~, J7 GND, U1 USBLC6-2SC6, U2 ATmega32U4-AU, Y1 Crystal_GND24

Commit message: housecleaning
Parts:
- LOGO5, LOGO6: value arisutea_logo -> QMK_Logo_Light; footprint arisutea:arisutea_logo -> 3x6_graphics:QMK_Logo_Light
Changed lines of the file:
@@
 P 10100 6100
 F 0 "LOGO5" H 10100 6300 50  0000 C CNN
-F 1 "arisutea_logo" H 10175 6474 50  0001 C CNN
-F 2 "arisutea:arisutea_logo" H 10100 6450 50  0001 C CNN
+F 1 "QMK_Logo_Light" H 10175 6474 50  0001 C CNN
+F 2 "3x6_graphics:QMK_Logo_Light" H 10100 6450 50  0001 C CNN
 F 3 "" H 10100 6450 50  0001 C CNN
 	1    10100 6100
@@
 P 10450 6100
 F 0 "LOGO6" H 10450 6300 50  0000 C CNN
-F 1 "arisutea_logo" H 10525 6474 50  0001 C CNN
-F 2 "arisutea:arisutea_logo" H 10450 6450 50  0001 C CNN
+F 1 "QMK_Logo_Light" H 10525 6474 50  0001 C CNN
+F 2 "3x6_graphics:QMK_Logo_Light" H 10450 6450 50  0001 C CNN
 F 3 "" H 10450 6450 50  0001 C CNN
 	1    10450 6100

Commit message: Initial upload of bluetooth version
Parts:
- removed C1, C2: 22pF, arisutea:C_0805_2012Metric_Pad1.18x1.45mm_HandSolder, symbol Device:C
- removed C3: 10uF, arisutea:C_0805_2012Metric_Pad1.18x1.45mm_HandSolder, symbol Device:C
- removed C4: 1uF (±10%), arisutea:C_0805_2012Metric_Pad1.18x1.45mm_HandSolder, symbol Device:C
- removed C5: 1uF, arisutea:C_0805_2012Metric_Pad1.18x1.45mm_HandSolder, symbol Device:C
- removed C6, C7, C8, C9: 0.1uF, arisutea:C_0805_2012Metric_Pad1.18x1.45mm_HandSolder, symbol Device:C
- removed J12: VCC, arisutea:PinHeader_1x01_P2.54mm_Vertical, symbol Connector_Generic:Conn_01x01
- removed J13: D+, arisutea:PinHeader_1x01_P2.54mm_Vertical, symbol Connector_Generic:Conn_01x01
- removed J14: D-, arisutea:PinHeader_1x01_P2.54mm_Vertical, symbol Connector_Generic:Conn_01x01
- removed J15, J7: GND, arisutea:PinHeader_1x01_P2.54mm_Vertical, symbol Connector_Generic:Conn_01x01
- removed J16: RGB, arisutea:PinHeader_1x03_P2.54mm_Vertical, symbol Connector_Generic:Conn_01x03
- removed J17: RGB_IN, arisutea:PinHeader_1x03_P2.54mm_Vertical, symbol Connector_Generic:Conn_01x03
- removed J18: RGB_OUT, arisutea:PinHeader_1x03_P2.54mm_Vertical, symbol Connector_Generic:Conn_01x03
- removed J2: MISO, arisutea:PinHeader_1x01_P2.54mm_Vertical, symbol Connector_Generic:Conn_01x01
- removed J3: +5V, arisutea:PinHeader_1x01_P2.54mm_Vertical, symbol Connector_Generic:Conn_01x01
- removed J4: SCK, arisutea:PinHeader_1x01_P2.54mm_Vertical, symbol Connector_Generic:Conn_01x01
- removed J5: MOSI, arisutea:PinHeader_1x01_P2.54mm_Vertical, symbol Connector_Generic:Conn_01x01
- removed J6: ~RES~, arisutea:PinHeader_1x01_P2.54mm_Vertical, symbol Connector_Generic:Conn_01x01
- removed LOGO3, LOGO4: arisutea_logo, Symbol:OSHW-Logo_5.7x6mm_SilkScreen, symbol arisutea-pcb-r1:arisutea_logo
- removed LOGO5, LOGO6: QMK_Logo_Light, 3x6_graphics:QMK_Logo_Light, symbol arisutea-pcb-r1:arisutea_logo
- removed R3, R4: 10K, arisutea:R_0805_2012Metric_Pad1.20x1.40mm_HandSolder, symbol Device:R
- removed R5, R6: 5k1, arisutea:R_0805_2012Metric_Pad1.20x1.40mm_HandSolder, symbol Device:R
- removed U1: USBLC6-2SC6, arisutea:SOT-23-6_Handsoldering, symbol arisutea-pcb-r1:USBLC6-2SC6-Power_Protection
- removed U2: ATmega32U4-AU, arisutea:TQFP-44_10x10mm_P0.8mm, symbol arisutea-pcb-r1:ATmega32U4-AU-MCU_Microchip_ATmega
- removed USB1: USB_C_HRO_TYPE-C-31-M-12-USB_Type-C, arisutea:USB_C_Receptacle_HRO_TYPE-C-31-M-12-HandSoldering, symbol arisutea-pcb-r1:USB_C_Receptacle_HRO_TYPE-C-31-M-12
- removed Y1: Crystal_GND24, arisutea:Crystal_SMD_TXC_7M-4Pin_3.2x2.5mm_HandSoldering, symbol Device:Crystal_GND24
- added BT1: Battery_Cell, arisutea-bt-pcb:Battery_Connector, symbol arisutea-bt-pcb:Battery_Cell
- added BT2: Battery_Cell, arisutea-bt-pcb:JST_PH_S2B-PH-K_1x02_P2.00mm_Horizontal, symbol arisutea-bt-pcb:Battery_Cell
- added C1: 4.7uF, arisutea-bt-pcb:C_0805_2012Metric_Pad1.18x1.45mm_HandSolder, symbol arisutea-bt-pcb:Device_C_Small
- added C2, C3: 1uF, arisutea-bt-pcb:C_0805_2012Metric_Pad1.18x1.45mm_HandSolder, symbol arisutea-bt-pcb:Device_C_Small
- added D1: 1N5819, arisutea-bt-pcb:D_SOD-123, symbol arisutea-bt-pcb:Device_D_Schottky_Small
- added J1: Conn_01x04, arisutea-bt-pcb:PinHeader_1x04_P2.54mm_Vertical, symbol arisutea-bt-pcb:Conn_01x04
- added LED1: PWR_LED, arisutea-bt-pcb:LED_IN-S124ARUW, symbol arisutea-bt-pcb:LED
- added LED5: BAT_LED, arisutea-bt-pcb:LED_IN-S124ARUW, symbol arisutea-bt-pcb:LED
- added Q1: AO3401A, arisutea-bt-pcb:SOT-23, symbol arisutea-bt-pcb:AO3401A
- added R1, R2: 5k1, arisutea-bt-pcb:R_0805_2012Metric_Pad1.20x1.40mm_HandSolder, symbol arisutea-bt-pcb:Device_R
- added R10: 1K, arisutea-bt-pcb:R_0805_2012Metric_Pad1.20x1.40mm_HandSolder, symbol arisutea-bt-pcb:Device_R
- added R5: 806K, arisutea-bt-pcb:R_0805_2012Metric_Pad1.20x1.40mm_HandSolder, symbol arisutea-bt-pcb:Device_R
- added R6: 2M, arisutea-bt-pcb:R_0805_2012Metric_Pad1.20x1.40mm_HandSolder, symbol arisutea-bt-pcb:Device_R
- added R7, R9: 10K, arisutea-bt-pcb:R_0805_2012Metric_Pad1.20x1.40mm_HandSolder, symbol arisutea-bt-pcb:Device_R
- added R8: 1k, arisutea-bt-pcb:R_0805_2012Metric_Pad1.20x1.40mm_HandSolder, symbol arisutea-bt-pcb:Device_R
- added SW67: Switch, arisutea-bt-pcb:OS102011MA1QN1, symbol arisutea-bt-pcb:Switch_SW_Push
- added U1: nRF52840_holyiot_18010, arisutea-bt-pcb:nRF52840_holyiot_18010_HS_simple, symbol arisutea-bt-pcb:nRF52840_holyiot_18010
- added U2: USBLC6-2SC6, arisutea-bt-pcb:SOT-23-6_Handsoldering, symbol arisutea-bt-pcb:USBLC6-2SC6-Power_Protection
- added U3: TP4504, arisutea-bt-pcb:SOT-23-5, symbol arisutea-bt-pcb:TP4504
- added U4: AP2112K-3.3, arisutea-bt-pcb:SOT-23-5, symbol arisutea-bt-pcb:AP2112K-3.3
- added USB1: HRO-TYPE-C-31-M-12-Type-C, arisutea-bt-pcb:USB_C_Receptacle_HRO_TYPE-C-31-M-12-HandSoldering, symbol arisutea-bt-pcb:HRO-TYPE-C-31-M-12-Type-C
- F1: footprint arisutea:Fuse_1206_3216Metric_Pad1.42x1.75mm_HandSolder -> arisutea-bt-pcb:Fuse_1206_3216Metric_Pad1.42x1.75mm_HandSolder; symbol Device:Polyfuse_Small -> arisutea-bt-pcb:Device_Polyfuse_Small
- H1, H2, H3, H4, H5, H6, H7, H8: footprint arisutea:Plated_Through_Hole_M2 -> arisutea-bt-pcb:Generic-Mounthole
- LED2: renamed from LED1; footprint arisutea:LED_IN-S124ARUW -> arisutea-bt-pcb:LED_IN-S124ARUW; symbol arisutea-pcb-r1:LED -> arisutea-bt-pcb:LED
- LED3: renamed from LED2; footprint arisutea:LED_IN-S124ARUW -> arisutea-bt-pcb:LED_IN-S124ARUW; symbol arisutea-pcb-r1:LED -> arisutea-bt-pcb:LED
- LED4: renamed from LED3; footprint arisutea:LED_IN-S124ARUW -> arisutea-bt-pcb:LED_IN-S124ARUW; symbol arisutea-pcb-r1:LED -> arisutea-bt-pcb:LED
- LOGO1, LOGO2: footprint arisutea:arisutea_logo -> arisutea-bt-pcb:arisutea_logo; symbol arisutea-pcb-r1:arisutea_logo -> arisutea-bt-pcb:arisutea_logo
- R11: renamed from R7; footprint arisutea:R_0805_2012Metric_Pad1.20x1.40mm_HandSolder -> arisutea-bt-pcb:R_0805_2012Metric_Pad1.20x1.40mm_HandSolder; symbol Device:R -> arisutea-bt-pcb:Device_R
- R12: renamed from R8; footprint arisutea:R_0805_2012Metric_Pad1.20x1.40mm_HandSolder -> arisutea-bt-pcb:R_0805_2012Metric_Pad1.20x1.40mm_HandSolder; symbol Device:R -> arisutea-bt-pcb:Device_R
- R13: renamed from R9; footprint arisutea:R_0805_2012Metric_Pad1.20x1.40mm_HandSolder -> arisutea-bt-pcb:R_0805_2012Metric_Pad1.20x1.40mm_HandSolder; symbol Device:R -> arisutea-bt-pcb:Device_R
- R3: renamed from R2; footprint arisutea:R_0805_2012Metric_Pad1.20x1.40mm_HandSolder -> arisutea-bt-pcb:R_0805_2012Metric_Pad1.20x1.40mm_HandSolder; symbol Device:R -> arisutea-bt-pcb:Device_R
- R4: renamed from R1; footprint arisutea:R_0805_2012Metric_Pad1.20x1.40mm_HandSolder -> arisutea-bt-pcb:R_0805_2012Metric_Pad1.20x1.40mm_HandSolder; symbol Device:R -> arisutea-bt-pcb:Device_R
- SWR1: footprint arisutea:SW_SPST_TL3342 -> arisutea-bt-pcb:SW_SPST_TL3342; symbol Switch:SW_Push -> arisutea-bt-pcb:Switch_SW_Push
Connections:
- net labels added: VBUS, VDD_nRF, bat_led, bat_volt, reset, swdclk, swdio, vbat, vbus_usb
- net labels removed: +5V, MISO, MOSI, RGB, RGB_5V, RGB_A, SCK, VCC, XTAL1, XTAL2, ~RES~
- wire segments 165 -> 131
- no-connect marks 3 -> 28
Other:
- note added: "Battery Management"
- note added: "USB Connection, ESD & Fuse"
- note added: "Voltage Reg & Reset Switch"
- moved on the sheet: F1, H2, H3, H4, H5, H6, H7, H8, R11, R12, R13, R3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
