File: matrix.sch (KiCad schematic (older format))
At the start: 132 parts, among them SW1 SW_Push, SW10 SW_Push, SW11 SW_Push, SW12 SW_Push, SW13 SW_Push, SW14 SW_Push, SW15 SW_Push, SW16 SW_Push, SW17 SW_Push, SW18 SW_Push, SW19 SW_Push, SW2 SW_Push, SW20 SW_Push, SW21 SW_Push, SW22 SW_Push, SW23 SW_Push, SW24 SW_Push, SW25 SW_Push, SW26 SW_Push, SW27 SW_Push, SW28 SW_Push, SW29 SW_Push, SW3 SW_Push, SW30 SW_Push, SW31 SW_Push, SW32 SW_Push, SW33 SW_Push, SW34 SW_Push, SW35 SW_Push, SW36 SW_Push, SW37 SW_Push, SW38 SW_Push, SW39 SW_Push, SW4 SW_Push, SW40 SW_Push, SW41 SW_Push, SW42 SW_Push, SW43 SW_Push, SW44 SW_Push, SW45 SW_Push, SW46 SW_Push, SW47 SW_Push, SW48 SW_Push, SW49 SW_Push, SW5 SW_Push, SW50 SW_Push, SW51 SW_Push, SW52 SW_Push, SW53 SW_Push, SW54 SW_Push, SW55 SW_Push, SW56 SW_Push, SW57 SW_Push, SW58 SW_Push, SW59 SW_Push, SW6 SW_Push, SW60 SW_Push, SW61 SW_Push, SW62 SW_Push, SW63 SW_Push, SW64 SW_Push, SW65 SW_Push, SW66 SW_Push, SW7 SW_Push, SW8 SW_Push, SW9 SW_Push

Commit message: housecleaning
Parts:
- SW1, SW10, SW11, SW12, SW13, SW14, SW15, SW16, SW17, SW18, SW19, SW2, SW20, SW21, SW22, SW23, SW24, SW25, SW26, SW27, SW28, SW29, SW3, SW30, SW31, SW32, SW33, SW34, SW35, SW36, SW37, SW38, SW39, SW4, SW40, SW41, SW42, SW43, SW44, SW45, SW46, SW47, SW48, SW49, SW5, SW50, SW51, SW52, SW53, SW54, SW55, SW56, SW57, SW58, SW59, SW6, SW60, SW61, SW62, SW63, SW64, SW65, SW66, SW7, SW8, SW9: symbol Switch:SW_Push -> arisutea-pcb-r1:Switch_SW_Keeb
Connections:
- net col0: now also SW1.1 (COL), SW2.1 (COL), SW3.1 (COL), SW4.1 (COL), SW5.1 (COL); no longer SW1.2 (ROW), SW2.2 (ROW), SW3.2 (ROW), SW4.2 (ROW), SW5.2 (ROW)
- net col1: now also SW6.1 (COL), SW7.1 (COL), SW8.1 (COL), SW9.1 (COL); no longer SW6.2 (ROW), SW7.2 (ROW), SW8.2 (ROW), SW9.2 (ROW)
- net col10: now also SW47.1 (COL), SW48.1 (COL), SW49.1 (COL), SW50.1 (COL); no longer SW47.2 (ROW), SW48.2 (ROW), SW49.2 (ROW), SW50.2 (ROW)
- net col11: now also SW51.1 (COL), SW52.1 (COL), SW53.1 (COL), SW54.1 (COL); no longer SW51.2 (ROW), SW52.2 (ROW), SW53.2 (ROW), SW54.2 (ROW)
- net col12: now also SW55.1 (COL), SW56.1 (COL), SW57.1 (COL), SW58.1 (COL); no longer SW55.2 (ROW), SW56.2 (ROW), SW57.2 (ROW), SW58.2 (ROW)
- net col13: now also SW59.1 (COL), SW60.1 (COL), SW61.1 (COL), SW62.1 (COL); no longer SW59.2 (ROW), SW60.2 (ROW), SW61.2 (ROW), SW62.2 (ROW)
- net col14: now also SW63.1 (COL), SW64.1 (COL), SW65.1 (COL), SW66.1 (COL); no longer SW63.2 (ROW), SW64.2 (ROW), SW65.2 (ROW), SW66.2 (ROW)
- net col2: now also SW10.1 (COL), SW11.1 (COL), SW12.1 (COL), SW13.1 (COL), SW14.1 (COL); no longer SW10.2 (ROW), SW11.2 (ROW), SW12.2 (ROW), SW13.2 (ROW), SW14.2 (ROW)
- net col3: now also SW15.1 (COL), SW16.1 (COL), SW17.1 (COL), SW18.1 (COL); no longer SW15.2 (ROW), SW16.2 (ROW), SW17.2 (ROW), SW18.2 (ROW)
- net col4: now also SW19.1 (COL), SW20.1 (COL), SW21.1 (COL), SW22.1 (COL), SW23.1 (COL); no longer SW19.2 (ROW), SW20.2 (ROW), SW21.2 (ROW), SW22.2 (ROW), SW23.2 (ROW)
- net col5: now also SW24.1 (COL), SW25.1 (COL), SW26.1 (COL), SW27.1 (COL), SW28.1 (COL); no longer SW24.2 (ROW), SW25.2 (ROW), SW26.2 (ROW), SW27.2 (ROW), SW28.2 (ROW)
- net col6: now also SW29.1 (COL), SW30.1 (COL), SW31.1 (COL), SW32.1 (COL); no longer SW29.2 (ROW), SW30.2 (ROW), SW31.2 (ROW), SW32.2 (ROW)
- net col7: now also SW33.1 (COL), SW34.1 (COL), SW35.1 (COL), SW36.1 (COL), SW37.1 (COL); no longer SW33.2 (ROW), SW34.2 (ROW), SW35.2 (ROW), SW36.2 (ROW), SW37.2 (ROW)
- net col8: now also SW38.1 (COL), SW39.1 (COL), SW40.1 (COL), SW41.1 (COL); no longer SW38.2 (ROW), SW39.2 (ROW), SW40.2 (ROW), SW41.2 (ROW)
- net col9: now also SW42.1 (COL), SW43.1 (COL), SW44.1 (COL), SW45.1 (COL), SW46.1 (COL); no longer SW42.2 (ROW), SW43.2 (ROW), SW44.2 (ROW), SW45.2 (ROW), SW46.2 (ROW)
- net at D1.2 (A): now also SW1.2 (ROW); no longer SW1.1 (COL)
- net at D6.2 (A): now also SW6.2 (ROW); no longer SW6.1 (COL)
- net at D2.2 (A): now also SW2.2 (ROW); no longer SW2.1 (COL)
- net at D7.2 (A): now also SW7.2 (ROW); no longer SW7.1 (COL)
- net at D3.2 (A): now also SW3.2 (ROW); no longer SW3.1 (COL)
- net at D4.2 (A): now also SW4.2 (ROW); no longer SW4.1 (COL)
- net at D5.2 (A): now also SW5.2 (ROW); no longer SW5.1 (COL)
- net at D8.2 (A): now also SW8.2 (ROW); no longer SW8.1 (COL)
- net at D9.2 (A): now also SW9.2 (ROW); no longer SW9.1 (COL)
- net at D10.2 (A): now also SW10.2 (ROW); no longer SW10.1 (COL)
- net at D11.2 (A): now also SW11.2 (ROW); no longer SW11.1 (COL)
- net at D12.2 (A): now also SW12.2 (ROW); no longer SW12.1 (COL)
- net at D13.2 (A): now also SW13.2 (ROW); no longer SW13.1 (COL)
- net at D14.2 (A): now also SW14.2 (ROW); no longer SW14.1 (COL)
- net at D15.2 (A): now also SW15.2 (ROW); no longer SW15.1 (COL)
- net at D16.2 (A): now also SW16.2 (ROW); no longer SW16.1 (COL)
- net at D17.2 (A): now also SW17.2 (ROW); no longer SW17.1 (COL)
- net at D18.2 (A): now also SW18.2 (ROW); no longer SW18.1 (COL)
- net at D19.2 (A): now also SW19.2 (ROW); no longer SW19.1 (COL)
- net at D20.2 (A): now also SW20.2 (ROW); no longer SW20.1 (COL)
- net at D21.2 (A): now also SW21.2 (ROW); no longer SW21.1 (COL)
- net at D22.2 (A): now also SW22.2 (ROW); no longer SW22.1 (COL)
- net at D23.2 (A): now also SW23.2 (ROW); no longer SW23.1 (COL)
- net at D24.2 (A): now also SW24.2 (ROW); no longer SW24.1 (COL)
- net at D25.2 (A): now also SW25.2 (ROW); no longer SW25.1 (COL)
- net at D26.2 (A): now also SW26.2 (ROW); no longer SW26.1 (COL)
- net at D27.2 (A): now also SW27.2 (ROW); no longer SW27.1 (COL)
- net at D28.2 (A): now also SW28.2 (ROW); no longer SW28.1 (COL)
- net at D29.2 (A): now also SW29.2 (ROW); no longer SW29.1 (COL)
- net at D30.2 (A): now also SW30.2 (ROW); no longer SW30.1 (COL)
- net at D31.2 (A): now also SW31.2 (ROW); no longer SW31.1 (COL)
- net at D32.2 (A): now also SW32.2 (ROW); no longer SW32.1 (COL)
- net at D33.2 (A): now also SW33.2 (ROW); no longer SW33.1 (COL)
- net at D34.2 (A): now also SW34.2 (ROW); no longer SW34.1 (COL)
- net at D35.2 (A): now also SW35.2 (ROW); no longer SW35.1 (COL)
- net at D36.2 (A): now also SW36.2 (ROW); no longer SW36.1 (COL)
- net at D37.2 (A): now also SW37.2 (ROW); no longer SW37.1 (COL)
- net at D38.2 (A): now also SW38.2 (ROW); no longer SW38.1 (COL)
- net at D39.2 (A): now also SW39.2 (ROW); no longer SW39.1 (COL)
- net at D40.2 (A): now also SW40.2 (ROW); no longer SW40.1 (COL)
- net at D41.2 (A): now also SW41.2 (ROW); no longer SW41.1 (COL)
- net at D42.2 (A): now also SW42.2 (ROW); no longer SW42.1 (COL)
- net at D43.2 (A): now also SW43.2 (ROW); no longer SW43.1 (COL)
- net at D44.2 (A): now also SW44.2 (ROW); no longer SW44.1 (COL)
- net at D45.2 (A): now also SW45.2 (ROW); no longer SW45.1 (COL)
- net at D46.2 (A): now also SW46.2 (ROW); no longer SW46.1 (COL)
- net at D47.2 (A): now also SW47.2 (ROW); no longer SW47.1 (COL)
- net at D48.2 (A): now also SW48.2 (ROW); no longer SW48.1 (COL)
- net at D49.2 (A): now also SW49.2 (ROW); no longer SW49.1 (COL)
- net at D50.2 (A): now also SW50.2 (ROW); no longer SW50.1 (COL)
- net at D51.2 (A): now also SW51.2 (ROW); no longer SW51.1 (COL)
- net at D52.2 (A): now also SW52.2 (ROW); no longer SW52.1 (COL)
- net at D53.2 (A): now also SW53.2 (ROW); no longer SW53.1 (COL)
- net at D54.2 (A): now also SW54.2 (ROW); no longer SW54.1 (COL)
- net at D55.2 (A): now also SW55.2 (ROW); no longer SW55.1 (COL)
- net at D56.2 (A): now also SW56.2 (ROW); no longer SW56.1 (COL)
- net at D57.2 (A): now also SW57.2 (ROW); no longer SW57.1 (COL)
- net at D58.2 (A): now also SW58.2 (ROW); no longer SW58.1 (COL)
- net at D59.2 (A): now also SW59.2 (ROW); no longer SW59.1 (COL)
- net at D60.2 (A): now also SW60.2 (ROW); no longer SW60.1 (COL)
- net at D61.2 (A): now also SW61.2 (ROW); no longer SW61.1 (COL)
- net at D62.2 (A): now also SW62.2 (ROW); no longer SW62.1 (COL)
- net at D63.2 (A): now also SW63.2 (ROW); no longer SW63.1 (COL)
- net at D64.2 (A): now also SW64.2 (ROW); no longer SW64.1 (COL)
- net at D65.2 (A): now also SW65.2 (ROW); no longer SW65.1 (COL)
- net at D66.2 (A): now also SW66.2 (ROW); no longer SW66.1 (COL)

Commit message: Initial upload of bluetooth version
Parts:
- D10: renamed from D38; footprint arisutea:D_SOD-123 -> arisutea-bt-pcb:D_SOD-123
- D11: renamed from D42; footprint arisutea:D_SOD-123 -> arisutea-bt-pcb:D_SOD-123
- D12: renamed from D47; footprint arisutea:D_SOD-123 -> arisutea-bt-pcb:D_SOD-123
- D13: renamed from D51; footprint arisutea:D_SOD-123 -> arisutea-bt-pcb:D_SOD-123
- D14: renamed from D55; footprint arisutea:D_SOD-123 -> arisutea-bt-pcb:D_SOD-123
- D15: renamed from D59; footprint arisutea:D_SOD-123 -> arisutea-bt-pcb:D_SOD-123
- D16: renamed from D2; footprint arisutea:D_SOD-123 -> arisutea-bt-pcb:D_SOD-123
- D17: renamed from D7; footprint arisutea:D_SOD-123 -> arisutea-bt-pcb:D_SOD-123
- D18: renamed from D11; footprint arisutea:D_SOD-123 -> arisutea-bt-pcb:D_SOD-123
- D19: renamed from D16; footprint arisutea:D_SOD-123 -> arisutea-bt-pcb:D_SOD-123
- D2: renamed from D1; footprint arisutea:D_SOD-123 -> arisutea-bt-pcb:D_SOD-123
- D20: footprint arisutea:D_SOD-123 -> arisutea-bt-pcb:D_SOD-123
- D21: renamed from D25; footprint arisutea:D_SOD-123 -> arisutea-bt-pcb:D_SOD-123
- D22: renamed from D30; footprint arisutea:D_SOD-123 -> arisutea-bt-pcb:D_SOD-123
- D23: renamed from D34; footprint arisutea:D_SOD-123 -> arisutea-bt-pcb:D_SOD-123
- D24: renamed from D39; footprint arisutea:D_SOD-123 -> arisutea-bt-pcb:D_SOD-123
- D25: renamed from D43; footprint arisutea:D_SOD-123 -> arisutea-bt-pcb:D_SOD-123
- D26: renamed from D48; footprint arisutea:D_SOD-123 -> arisutea-bt-pcb:D_SOD-123
- D27: renamed from D52; footprint arisutea:D_SOD-123 -> arisutea-bt-pcb:D_SOD-123
- D28: renamed from D56; footprint arisutea:D_SOD-123 -> arisutea-bt-pcb:D_SOD-123
- D29: renamed from D60; footprint arisutea:D_SOD-123 -> arisutea-bt-pcb:D_SOD-123
- D3: renamed from D6; footprint arisutea:D_SOD-123 -> arisutea-bt-pcb:D_SOD-123
- D30: renamed from D63; footprint arisutea:D_SOD-123 -> arisutea-bt-pcb:D_SOD-123
- D31: renamed from D3; footprint arisutea:D_SOD-123 -> arisutea-bt-pcb:D_SOD-123
- D32: renamed from D8; footprint arisutea:D_SOD-123 -> arisutea-bt-pcb:D_SOD-123
- D33: renamed from D12; footprint arisutea:D_SOD-123 -> arisutea-bt-pcb:D_SOD-123
- D34: renamed from D17; footprint arisutea:D_SOD-123 -> arisutea-bt-pcb:D_SOD-123
- D35: renamed from D21; footprint arisutea:D_SOD-123 -> arisutea-bt-pcb:D_SOD-123
- D36: renamed from D26; footprint arisutea:D_SOD-123 -> arisutea-bt-pcb:D_SOD-123
- D37: renamed from D31; footprint arisutea:D_SOD-123 -> arisutea-bt-pcb:D_SOD-123
- D38: renamed from D35; footprint arisutea:D_SOD-123 -> arisutea-bt-pcb:D_SOD-123
- D39: renamed from D40; footprint arisutea:D_SOD-123 -> arisutea-bt-pcb:D_SOD-123
- D4: renamed from D10; footprint arisutea:D_SOD-123 -> arisutea-bt-pcb:D_SOD-123
- D40: renamed from D44; footprint arisutea:D_SOD-123 -> arisutea-bt-pcb:D_SOD-123
- D41: renamed from D49; footprint arisutea:D_SOD-123 -> arisutea-bt-pcb:D_SOD-123
- D42: renamed from D53; footprint arisutea:D_SOD-123 -> arisutea-bt-pcb:D_SOD-123
- D43: renamed from D57; footprint arisutea:D_SOD-123 -> arisutea-bt-pcb:D_SOD-123
- D44: renamed from D64; footprint arisutea:D_SOD-123 -> arisutea-bt-pcb:D_SOD-123
- D45: renamed from D4; footprint arisutea:D_SOD-123 -> arisutea-bt-pcb:D_SOD-123
- D46: renamed from D9; footprint arisutea:D_SOD-123 -> arisutea-bt-pcb:D_SOD-123
- D47: renamed from D13; footprint arisutea:D_SOD-123 -> arisutea-bt-pcb:D_SOD-123
- D48: renamed from D18; footprint arisutea:D_SOD-123 -> arisutea-bt-pcb:D_SOD-123
- D49: renamed from D22; footprint arisutea:D_SOD-123 -> arisutea-bt-pcb:D_SOD-123
- D5: renamed from D15; footprint arisutea:D_SOD-123 -> arisutea-bt-pcb:D_SOD-123
- D50: renamed from D27; footprint arisutea:D_SOD-123 -> arisutea-bt-pcb:D_SOD-123
- D51: renamed from D32; footprint arisutea:D_SOD-123 -> arisutea-bt-pcb:D_SOD-123
- D52: renamed from D36; footprint arisutea:D_SOD-123 -> arisutea-bt-pcb:D_SOD-123
- D53: renamed from D41; footprint arisutea:D_SOD-123 -> arisutea-bt-pcb:D_SOD-123
- D54: renamed from D45; footprint arisutea:D_SOD-123 -> arisutea-bt-pcb:D_SOD-123
- D55: renamed from D50; footprint arisutea:D_SOD-123 -> arisutea-bt-pcb:D_SOD-123
- D56: renamed from D54; footprint arisutea:D_SOD-123 -> arisutea-bt-pcb:D_SOD-123
- D57: renamed from D61; footprint arisutea:D_SOD-123 -> arisutea-bt-pcb:D_SOD-123
- D58: renamed from D65; footprint arisutea:D_SOD-123 -> arisutea-bt-pcb:D_SOD-123
- D59: renamed from D5; footprint arisutea:D_SOD-123 -> arisutea-bt-pcb:D_SOD-123
- D6: renamed from D19; footprint arisutea:D_SOD-123 -> arisutea-bt-pcb:D_SOD-123
- D60: renamed from D14; footprint arisutea:D_SOD-123 -> arisutea-bt-pcb:D_SOD-123
- D61: renamed from D23; footprint arisutea:D_SOD-123 -> arisutea-bt-pcb:D_SOD-123
- D62: renamed from D28; footprint arisutea:D_SOD-123 -> arisutea-bt-pcb:D_SOD-123
- D63: renamed from D37; footprint arisutea:D_SOD-123 -> arisutea-bt-pcb:D_SOD-123
- D64: renamed from D46; footprint arisutea:D_SOD-123 -> arisutea-bt-pcb:D_SOD-123
- D65: renamed from D58; footprint arisutea:D_SOD-123 -> arisutea-bt-pcb:D_SOD-123
- D66: renamed from D62; footprint arisutea:D_SOD-123 -> arisutea-bt-pcb:D_SOD-123
- D67: renamed from D66; footprint arisutea:D_SOD-123 -> arisutea-bt-pcb:D_SOD-123
- D7: renamed from D24; footprint arisutea:D_SOD-123 -> arisutea-bt-pcb:D_SOD-123
- D8: renamed from D29; footprint arisutea:D_SOD-123 -> arisutea-bt-pcb:D_SOD-123
- D9: renamed from D33; footprint arisutea:D_SOD-123 -> arisutea-bt-pcb:D_SOD-123
- SW1, SW66: footprint arisutea:SW_Hotswap_Kailh_1.00u -> arisutea-bt-pcb:SW_Hotswap_Kailh_1.00u; symbol arisutea-pcb-r1:Switch_SW_Keeb -> arisutea-bt-pcb:Switch_SW_Keeb
- SW10: renamed from SW42; footprint arisutea:SW_Hotswap_Kailh_1.00u -> arisutea-bt-pcb:SW_Hotswap_Kailh_1.00u; symbol arisutea-pcb-r1:Switch_SW_Keeb -> arisutea-bt-pcb:Switch_SW_Keeb
- SW11: renamed from SW47; footprint arisutea:SW_Hotswap_Kailh_1.00u -> arisutea-bt-pcb:SW_Hotswap_Kailh_1.00u; symbol arisutea-pcb-r1:Switch_SW_Keeb -> arisutea-bt-pcb:Switch_SW_Keeb
- SW12: renamed from SW51; footprint arisutea:SW_Hotswap_Kailh_1.00u -> arisutea-bt-pcb:SW_Hotswap_Kailh_1.00u; symbol arisutea-pcb-r1:Switch_SW_Keeb -> arisutea-bt-pcb:Switch_SW_Keeb
- SW13: renamed from SW55; footprint arisutea:SW_Hotswap_Kailh_1.00u -> arisutea-bt-pcb:SW_Hotswap_Kailh_1.00u; symbol arisutea-pcb-r1:Switch_SW_Keeb -> arisutea-bt-pcb:Switch_SW_Keeb
- SW14: renamed from SW59; footprint arisutea:SW_Hotswap_Kailh_2.00u -> arisutea-bt-pcb:SW_Hotswap_Kailh_2.00u; symbol arisutea-pcb-r1:Switch_SW_Keeb -> arisutea-bt-pcb:Switch_SW_Keeb
- SW15: renamed from SW2; footprint arisutea:SW_Hotswap_Kailh_1.50u -> arisutea-bt-pcb:SW_Hotswap_Kailh_1.50u; symbol arisutea-pcb-r1:Switch_SW_Keeb -> arisutea-bt-pcb:Switch_SW_Keeb
- SW16: renamed from SW7; footprint arisutea:SW_Hotswap_Kailh_1.00u -> arisutea-bt-pcb:SW_Hotswap_Kailh_1.00u; symbol arisutea-pcb-r1:Switch_SW_Keeb -> arisutea-bt-pcb:Switch_SW_Keeb
- SW17: renamed from SW11; footprint arisutea:SW_Hotswap_Kailh_1.00u -> arisutea-bt-pcb:SW_Hotswap_Kailh_1.00u; symbol arisutea-pcb-r1:Switch_SW_Keeb -> arisutea-bt-pcb:Switch_SW_Keeb
- SW18: renamed from SW16; footprint arisutea:SW_Hotswap_Kailh_1.00u -> arisutea-bt-pcb:SW_Hotswap_Kailh_1.00u; symbol arisutea-pcb-r1:Switch_SW_Keeb -> arisutea-bt-pcb:Switch_SW_Keeb
- SW19: renamed from SW20; footprint arisutea:SW_Hotswap_Kailh_1.00u -> arisutea-bt-pcb:SW_Hotswap_Kailh_1.00u; symbol arisutea-pcb-r1:Switch_SW_Keeb -> arisutea-bt-pcb:Switch_SW_Keeb
- SW2: renamed from SW6; footprint arisutea:SW_Hotswap_Kailh_1.00u -> arisutea-bt-pcb:SW_Hotswap_Kailh_1.00u; symbol arisutea-pcb-r1:Switch_SW_Keeb -> arisutea-bt-pcb:Switch_SW_Keeb
- SW20: renamed from SW25; footprint arisutea:SW_Hotswap_Kailh_1.00u -> arisutea-bt-pcb:SW_Hotswap_Kailh_1.00u; symbol arisutea-pcb-r1:Switch_SW_Keeb -> arisutea-bt-pcb:Switch_SW_Keeb
- SW21: renamed from SW30; footprint arisutea:SW_Hotswap_Kailh_1.00u -> arisutea-bt-pcb:SW_Hotswap_Kailh_1.00u; symbol arisutea-pcb-r1:Switch_SW_Keeb -> arisutea-bt-pcb:Switch_SW_Keeb
- SW22: renamed from SW34; footprint arisutea:SW_Hotswap_Kailh_1.00u -> arisutea-bt-pcb:SW_Hotswap_Kailh_1.00u; symbol arisutea-pcb-r1:Switch_SW_Keeb -> arisutea-bt-pcb:Switch_SW_Keeb
- SW23: renamed from SW39; footprint arisutea:SW_Hotswap_Kailh_1.00u -> arisutea-bt-pcb:SW_Hotswap_Kailh_1.00u; symbol arisutea-pcb-r1:Switch_SW_Keeb -> arisutea-bt-pcb:Switch_SW_Keeb
- SW24: renamed from SW43; footprint arisutea:SW_Hotswap_Kailh_1.00u -> arisutea-bt-pcb:SW_Hotswap_Kailh_1.00u; symbol arisutea-pcb-r1:Switch_SW_Keeb -> arisutea-bt-pcb:Switch_SW_Keeb
- SW25: renamed from SW48; footprint arisutea:SW_Hotswap_Kailh_1.00u -> arisutea-bt-pcb:SW_Hotswap_Kailh_1.00u; symbol arisutea-pcb-r1:Switch_SW_Keeb -> arisutea-bt-pcb:Switch_SW_Keeb
- SW26: renamed from SW52; footprint arisutea:SW_Hotswap_Kailh_1.00u -> arisutea-bt-pcb:SW_Hotswap_Kailh_1.00u; symbol arisutea-pcb-r1:Switch_SW_Keeb -> arisutea-bt-pcb:Switch_SW_Keeb
- SW27: renamed from SW56; footprint arisutea:SW_Hotswap_Kailh_1.00u -> arisutea-bt-pcb:SW_Hotswap_Kailh_1.00u; symbol arisutea-pcb-r1:Switch_SW_Keeb -> arisutea-bt-pcb:Switch_SW_Keeb
- SW28: renamed from SW60; footprint arisutea:SW_Hotswap_Kailh_1.50u -> arisutea-bt-pcb:SW_Hotswap_Kailh_1.50u; symbol arisutea-pcb-r1:Switch_SW_Keeb -> arisutea-bt-pcb:Switch_SW_Keeb
- SW29: renamed from SW63; footprint arisutea:SW_Hotswap_Kailh_1.00u -> arisutea-bt-pcb:SW_Hotswap_Kailh_1.00u; symbol arisutea-pcb-r1:Switch_SW_Keeb -> arisutea-bt-pcb:Switch_SW_Keeb
- SW3: renamed from SW10; footprint arisutea:SW_Hotswap_Kailh_1.00u -> arisutea-bt-pcb:SW_Hotswap_Kailh_1.00u; symbol arisutea-pcb-r1:Switch_SW_Keeb -> arisutea-bt-pcb:Switch_SW_Keeb
- SW30: renamed from SW3; footprint arisutea:SW_Hotswap_Kailh_1.75u -> arisutea-bt-pcb:SW_Hotswap_Kailh_1.75u; symbol arisutea-pcb-r1:Switch_SW_Keeb -> arisutea-bt-pcb:Switch_SW_Keeb
- SW31: renamed from SW8; footprint arisutea:SW_Hotswap_Kailh_1.00u -> arisutea-bt-pcb:SW_Hotswap_Kailh_1.00u; symbol arisutea-pcb-r1:Switch_SW_Keeb -> arisutea-bt-pcb:Switch_SW_Keeb
- SW32: renamed from SW12; footprint arisutea:SW_Hotswap_Kailh_1.00u -> arisutea-bt-pcb:SW_Hotswap_Kailh_1.00u; symbol arisutea-pcb-r1:Switch_SW_Keeb -> arisutea-bt-pcb:Switch_SW_Keeb
- SW33: renamed from SW17; footprint arisutea:SW_Hotswap_Kailh_1.00u -> arisutea-bt-pcb:SW_Hotswap_Kailh_1.00u; symbol arisutea-pcb-r1:Switch_SW_Keeb -> arisutea-bt-pcb:Switch_SW_Keeb
- SW34: renamed from SW21; footprint arisutea:SW_Hotswap_Kailh_1.00u -> arisutea-bt-pcb:SW_Hotswap_Kailh_1.00u; symbol arisutea-pcb-r1:Switch_SW_Keeb -> arisutea-bt-pcb:Switch_SW_Keeb
- SW35: renamed from SW26; footprint arisutea:SW_Hotswap_Kailh_1.00u -> arisutea-bt-pcb:SW_Hotswap_Kailh_1.00u; symbol arisutea-pcb-r1:Switch_SW_Keeb -> arisutea-bt-pcb:Switch_SW_Keeb
- SW36: renamed from SW31; footprint arisutea:SW_Hotswap_Kailh_1.00u -> arisutea-bt-pcb:SW_Hotswap_Kailh_1.00u; symbol arisutea-pcb-r1:Switch_SW_Keeb -> arisutea-bt-pcb:Switch_SW_Keeb
- SW37: renamed from SW35; footprint arisutea:SW_Hotswap_Kailh_1.00u -> arisutea-bt-pcb:SW_Hotswap_Kailh_1.00u; symbol arisutea-pcb-r1:Switch_SW_Keeb -> arisutea-bt-pcb:Switch_SW_Keeb
- SW38: renamed from SW40; footprint arisutea:SW_Hotswap_Kailh_1.00u -> arisutea-bt-pcb:SW_Hotswap_Kailh_1.00u; symbol arisutea-pcb-r1:Switch_SW_Keeb -> arisutea-bt-pcb:Switch_SW_Keeb
- SW39: renamed from SW44; footprint arisutea:SW_Hotswap_Kailh_1.00u -> arisutea-bt-pcb:SW_Hotswap_Kailh_1.00u; symbol arisutea-pcb-r1:Switch_SW_Keeb -> arisutea-bt-pcb:Switch_SW_Keeb
- SW4: renamed from SW15; footprint arisutea:SW_Hotswap_Kailh_1.00u -> arisutea-bt-pcb:SW_Hotswap_Kailh_1.00u; symbol arisutea-pcb-r1:Switch_SW_Keeb -> arisutea-bt-pcb:Switch_SW_Keeb
- SW40: renamed from SW49; footprint arisutea:SW_Hotswap_Kailh_1.00u -> arisutea-bt-pcb:SW_Hotswap_Kailh_1.00u; symbol arisutea-pcb-r1:Switch_SW_Keeb -> arisutea-bt-pcb:Switch_SW_Keeb
- SW41: renamed from SW53; footprint arisutea:SW_Hotswap_Kailh_1.00u -> arisutea-bt-pcb:SW_Hotswap_Kailh_1.00u; symbol arisutea-pcb-r1:Switch_SW_Keeb -> arisutea-bt-pcb:Switch_SW_Keeb
- SW42: renamed from SW57; footprint arisutea:SW_Hotswap_Kailh_2.25u_RevStab -> arisutea-bt-pcb:SW_Hotswap_Kailh_2.25u_RevStab; symbol arisutea-pcb-r1:Switch_SW_Keeb -> arisutea-bt-pcb:Switch_SW_Keeb
- SW43: renamed from SW64; footprint arisutea:SW_Hotswap_Kailh_1.00u -> arisutea-bt-pcb:SW_Hotswap_Kailh_1.00u; symbol arisutea-pcb-r1:Switch_SW_Keeb -> arisutea-bt-pcb:Switch_SW_Keeb
- SW44: renamed from SW4; footprint arisutea:SW_Hotswap_Kailh_2.25u -> arisutea-bt-pcb:SW_Hotswap_Kailh_2.25u; symbol arisutea-pcb-r1:Switch_SW_Keeb -> arisutea-bt-pcb:Switch_SW_Keeb
- SW45: renamed from SW9; footprint arisutea:SW_Hotswap_Kailh_1.00u -> arisutea-bt-pcb:SW_Hotswap_Kailh_1.00u; symbol arisutea-pcb-r1:Switch_SW_Keeb -> arisutea-bt-pcb:Switch_SW_Keeb
- SW46: renamed from SW13; footprint arisutea:SW_Hotswap_Kailh_1.00u -> arisutea-bt-pcb:SW_Hotswap_Kailh_1.00u; symbol arisutea-pcb-r1:Switch_SW_Keeb -> arisutea-bt-pcb:Switch_SW_Keeb
- SW47: renamed from SW18; footprint arisutea:SW_Hotswap_Kailh_1.00u -> arisutea-bt-pcb:SW_Hotswap_Kailh_1.00u; symbol arisutea-pcb-r1:Switch_SW_Keeb -> arisutea-bt-pcb:Switch_SW_Keeb
- SW48: renamed from SW22; footprint arisutea:SW_Hotswap_Kailh_1.00u -> arisutea-bt-pcb:SW_Hotswap_Kailh_1.00u; symbol arisutea-pcb-r1:Switch_SW_Keeb -> arisutea-bt-pcb:Switch_SW_Keeb
- SW49: renamed from SW27; footprint arisutea:SW_Hotswap_Kailh_1.00u -> arisutea-bt-pcb:SW_Hotswap_Kailh_1.00u; symbol arisutea-pcb-r1:Switch_SW_Keeb -> arisutea-bt-pcb:Switch_SW_Keeb
- SW5: renamed from SW19; footprint arisutea:SW_Hotswap_Kailh_1.00u -> arisutea-bt-pcb:SW_Hotswap_Kailh_1.00u; symbol arisutea-pcb-r1:Switch_SW_Keeb -> arisutea-bt-pcb:Switch_SW_Keeb
- SW50: renamed from SW32; footprint arisutea:SW_Hotswap_Kailh_1.00u -> arisutea-bt-pcb:SW_Hotswap_Kailh_1.00u; symbol arisutea-pcb-r1:Switch_SW_Keeb -> arisutea-bt-pcb:Switch_SW_Keeb
- SW51: renamed from SW36; footprint arisutea:SW_Hotswap_Kailh_1.00u -> arisutea-bt-pcb:SW_Hotswap_Kailh_1.00u; symbol arisutea-pcb-r1:Switch_SW_Keeb -> arisutea-bt-pcb:Switch_SW_Keeb
- SW52: renamed from SW41; footprint arisutea:SW_Hotswap_Kailh_1.00u -> arisutea-bt-pcb:SW_Hotswap_Kailh_1.00u; symbol arisutea-pcb-r1:Switch_SW_Keeb -> arisutea-bt-pcb:Switch_SW_Keeb
- SW53: renamed from SW45; footprint arisutea:SW_Hotswap_Kailh_1.00u -> arisutea-bt-pcb:SW_Hotswap_Kailh_1.00u; symbol arisutea-pcb-r1:Switch_SW_Keeb -> arisutea-bt-pcb:Switch_SW_Keeb
- SW54: renamed from SW50; footprint arisutea:SW_Hotswap_Kailh_1.00u -> arisutea-bt-pcb:SW_Hotswap_Kailh_1.00u; symbol arisutea-pcb-r1:Switch_SW_Keeb -> arisutea-bt-pcb:Switch_SW_Keeb
- SW55: renamed from SW54; footprint arisutea:SW_Hotswap_Kailh_1.75u -> arisutea-bt-pcb:SW_Hotswap_Kailh_1.75u; symbol arisutea-pcb-r1:Switch_SW_Keeb -> arisutea-bt-pcb:Switch_SW_Keeb
- SW56: renamed from SW61; footprint arisutea:SW_Hotswap_Kailh_1.00u -> arisutea-bt-pcb:SW_Hotswap_Kailh_1.00u; symbol arisutea-pcb-r1:Switch_SW_Keeb -> arisutea-bt-pcb:Switch_SW_Keeb
- SW57: renamed from SW65; footprint arisutea:SW_Hotswap_Kailh_1.00u -> arisutea-bt-pcb:SW_Hotswap_Kailh_1.00u; symbol arisutea-pcb-r1:Switch_SW_Keeb -> arisutea-bt-pcb:Switch_SW_Keeb
- SW58: renamed from SW5; footprint arisutea:SW_Hotswap_Kailh_1.50u -> arisutea-bt-pcb:SW_Hotswap_Kailh_1.50u; symbol arisutea-pcb-r1:Switch_SW_Keeb -> arisutea-bt-pcb:Switch_SW_Keeb
- SW59: renamed from SW14; footprint arisutea:SW_Hotswap_Kailh_1.00u -> arisutea-bt-pcb:SW_Hotswap_Kailh_1.00u; symbol arisutea-pcb-r1:Switch_SW_Keeb -> arisutea-bt-pcb:Switch_SW_Keeb
- SW6: renamed from SW24; footprint arisutea:SW_Hotswap_Kailh_1.00u -> arisutea-bt-pcb:SW_Hotswap_Kailh_1.00u; symbol arisutea-pcb-r1:Switch_SW_Keeb -> arisutea-bt-pcb:Switch_SW_Keeb
- SW60: renamed from SW23; footprint arisutea:SW_Hotswap_Kailh_2.00u_RevStab -> arisutea-bt-pcb:SW_Hotswap_Kailh_2.00u_RevStab; symbol arisutea-pcb-r1:Switch_SW_Keeb -> arisutea-bt-pcb:Switch_SW_Keeb
- SW61: renamed from SW28; footprint arisutea:SW_Hotswap_Kailh_1.00u -> arisutea-bt-pcb:SW_Hotswap_Kailh_1.00u; symbol arisutea-pcb-r1:Switch_SW_Keeb -> arisutea-bt-pcb:Switch_SW_Keeb
- SW62: renamed from SW37; footprint arisutea:SW_Hotswap_Kailh_2.75u_RevStab -> arisutea-bt-pcb:SW_Hotswap_Kailh_2.75u_RevStab; symbol arisutea-pcb-r1:Switch_SW_Keeb -> arisutea-bt-pcb:Switch_SW_Keeb
- SW63: renamed from SW46; footprint arisutea:SW_Hotswap_Kailh_1.00u -> arisutea-bt-pcb:SW_Hotswap_Kailh_1.00u; symbol arisutea-pcb-r1:Switch_SW_Keeb -> arisutea-bt-pcb:Switch_SW_Keeb
- SW64: renamed from SW58; footprint arisutea:SW_Hotswap_Kailh_1.00u -> arisutea-bt-pcb:SW_Hotswap_Kailh_1.00u; symbol arisutea-pcb-r1:Switch_SW_Keeb -> arisutea-bt-pcb:Switch_SW_Keeb
- SW65: renamed from SW62; footprint arisutea:SW_Hotswap_Kailh_1.00u -> arisutea-bt-pcb:SW_Hotswap_Kailh_1.00u; symbol arisutea-pcb-r1:Switch_SW_Keeb -> arisutea-bt-pcb:Switch_SW_Keeb
- SW7: renamed from SW29; footprint arisutea:SW_Hotswap_Kailh_1.00u -> arisutea-bt-pcb:SW_Hotswap_Kailh_1.00u; symbol arisutea-pcb-r1:Switch_SW_Keeb -> arisutea-bt-pcb:Switch_SW_Keeb
- SW8: renamed from SW33; footprint arisutea:SW_Hotswap_Kailh_1.00u -> arisutea-bt-pcb:SW_Hotswap_Kailh_1.00u; symbol arisutea-pcb-r1:Switch_SW_Keeb -> arisutea-bt-pcb:Switch_SW_Keeb
- SW9: renamed from SW38; footprint arisutea:SW_Hotswap_Kailh_1.00u -> arisutea-bt-pcb:SW_Hotswap_Kailh_1.00u; symbol arisutea-pcb-r1:Switch_SW_Keeb -> arisutea-bt-pcb:Switch_SW_Keeb
